Commit message: comitting all urdf , coord changes

File: niryo_one_description/urdf/niryo_one.urdf (robot description, URDF)
Before this commit: robot niryo_one, 9 links, 8 joints
Joints:
- joint hand_gripper_joint: origin xyz=0 0 0.0 rpy=-1.5707963268 -1.5707963268 0 -> xyz=0 -0.014 0.1115 rpy=0 3.14159265359 -1.5707963268

File: niryo_one_description/urdf/niryo_one.urdf.xacro (robot description, xacro)
@@ -27,5 +27,6 @@
     <xacro:property name="distance_wrist_hand_y" value="0" />
     <!-- not yet implemented, for now -->
-    <xacro:property name="distance_hand_gripper" value="0.00" />
+    <xacro:property name="distance_hand_gripper_z" value="0.1115" />
+    <xacro:property name="distance_hand_gripper_y" value="-0.014" />
 	<xacro:property name="thickness_arm_axis" value="0.052" />
 	<xacro:property name="thickness_forearm_axis" value="0.048" />
@@ -218,5 +219,5 @@
         <parent link="hand_link" />
         <child link="gripper_link" />
-        <origin xyz="0 0 ${distance_hand_gripper}" rpy="${-PI/2} ${-PI/2} 0" />
+        <origin xyz="0 ${distance_hand_gripper_y} ${distance_hand_gripper_z}" rpy="0 ${PI} -${PI/2}" />
 	</joint>
 </robot>

File: niryo_one_description/urdf/without_mesh_niryo_one.urdf (robot description, URDF)
Before this commit: robot niryo_one, 9 links, 8 joints
Joints:
- joint hand_gripper_joint: origin xyz=0 0 0.0 rpy=-1.5707963268 -1.5707963268 0 -> xyz=0 0 0.035 rpy=0 3.14159265359 -1.5707963268

File: niryo_one_description/urdf/without_mesh_niryo_one.urdf.xacro (robot description, xacro)
@@ -27,5 +27,5 @@
     <xacro:property name="distance_wrist_hand_y" value="0" />
     <!-- not yet implemented, tools are handled separately -->
-    <xacro:property name="distance_hand_gripper" value="0.00" />
+    <xacro:property name="distance_hand_gripper" value="0.035" />
 	<xacro:property name="thickness_arm_axis" value="0.052" />
 	<xacro:property name="thickness_forearm_axis" value="0.048" />
@@ -112,5 +112,5 @@
         <parent link="hand_link" />
         <child link="gripper_link" />
-        <origin xyz="0 0 ${distance_hand_gripper}" rpy="${-PI/2} ${-PI/2} 0" />
+        <origin xyz="0 0 ${distance_hand_gripper}" rpy="0 ${PI} -${PI/2}" />
 	</joint>
 </robot>

Commit message: adding support for quaternian pose

File: niryo_one_description/urdf/niryo_one.urdf (robot description, URDF)
Before this commit: robot niryo_one, 9 links, 8 joints
Joints:
- joint hand_gripper_joint: origin xyz=0 -0.014 0.1115 rpy=0 3.14159265359 -1.5707963268 -> xyz=0 0 0.0 rpy=-1.5707963268 -1.5707963268 0

File: niryo_one_description/urdf/niryo_one.urdf.xacro (robot description, xacro)
@@ -27,6 +27,5 @@
     <xacro:property name="distance_wrist_hand_y" value="0" />
     <!-- not yet implemented, for now -->
-    <xacro:property name="distance_hand_gripper_z" value="0.1115" />
-    <xacro:property name="distance_hand_gripper_y" value="-0.014" />
+    <xacro:property name="distance_hand_gripper" value="0.00" />
 	<xacro:property name="thickness_arm_axis" value="0.052" />
 	<xacro:property name="thickness_forearm_axis" value="0.048" />
@@ -219,5 +218,5 @@
         <parent link="hand_link" />
         <child link="gripper_link" />
-        <origin xyz="0 ${distance_hand_gripper_y} ${distance_hand_gripper_z}" rpy="0 ${PI} -${PI/2}" />
+        <origin xyz="0 0 ${distance_hand_gripper}" rpy="${-PI/2} ${-PI/2} 0" />
 	</joint>
 </robot>

File: niryo_one_description/urdf/without_mesh_niryo_one.urdf (robot description, URDF)
Before this commit: robot niryo_one, 9 links, 8 joints
Joints:
- joint hand_gripper_joint: origin xyz=0 0 0.035 rpy=0 3.14159265359 -1.5707963268 -> xyz=0 0 0.0 rpy=-1.5707963268 -1.5707963268 0

File: niryo_one_description/urdf/without_mesh_niryo_one.urdf.xacro (robot description, xacro)
@@ -27,5 +27,5 @@
     <xacro:property name="distance_wrist_hand_y" value="0" />
     <!-- not yet implemented, tools are handled separately -->
-    <xacro:property name="distance_hand_gripper" value="0.035" />
+    <xacro:property name="distance_hand_gripper" value="0.00" />
 	<xacro:property name="thickness_arm_axis" value="0.052" />
 	<xacro:property name="thickness_forearm_axis" value="0.048" />
@@ -112,5 +112,5 @@
         <parent link="hand_link" />
         <child link="gripper_link" />
-        <origin xyz="0 0 ${distance_hand_gripper}" rpy="0 ${PI} -${PI/2}" />
+        <origin xyz="0 0 ${distance_hand_gripper}" rpy="${-PI/2} ${-PI/2} 0" />
 	</joint>
 </robot>
