Commit message: create gazebo aspects of niryo and add it to urdf file

File: niryo_one_description/urdf/v1/niryo_one.urdf (robot description, URDF)
Before this commit: robot niryo_one, 9 links, 8 joints
Links:
- link arm_link: mass None -> 0.5
- link base_link: mass None -> 1.3
- link elbow_link: mass None -> 0.4
- link forearm_link: mass None -> 0.3
- link hand_link: mass None -> 0.1
- link shoulder_link: mass None -> 0.6
- link wrist_link: mass None -> 0.2

File: niryo_one_description/urdf/v1/niryo_one.urdf.xacro (robot description, xacro)
@@ -43,6 +43,15 @@
     <xacro:property name="limit_low_hand_rotation" value="-2.57" />
     <xacro:property name="limit_up_hand_rotation" value="2.57" />
+    <xacro:include filename="$(find niryo_one_description)/urdf/v1/niryo_one.gazebo.xacro" />
 	<!-- Links -->
     <link name="ground_link"/>
+		<inertial>
+			<origin xyz="0 0 0" rpy="0 0 0"/>
+      		<mass value="1"/>
+      		<inertia
+        		ixx="0.0" ixy="0.0" ixz="0.0"
+        		iyy="0.0" iyz="0.0"
+        		izz="0.0"/>
+    	</inertial>
     <link name="base_link">
 		<visual>
@@ -61,4 +70,12 @@
             </geometry>
         </collision>
+		<inertial>
+      		<origin xyz="0 0 0" rpy="0 0 0"/>
+      		<mass value="1.3"/>
+      		<inertia
+        		ixx="0.0" ixy="0.0" ixz="0.0"
+        		iyy="0.0" iyz="0.0"
+        		izz="0.0"/>
+    	</inertial>
 	</link>
     <link name="shoulder_link">
@@ -78,4 +95,12 @@
             </geometry>
         </collision>
+		<inertial>
+      		<origin xyz="0 0 0" rpy="0 0 0"/>
+      		<mass value="0.6"/>
+      		<inertia
+        		ixx="1.0" ixy="0.0" ixz="0.0"
+        		iyy="1.0" iyz="0.0"
+        		izz="1.0"/>
+    	</inertial>
 	</link>
     <link name="arm_link">
@@ -95,4 +120,12 @@
             </geometry>
         </collision>
+		<inertial>
+      		<origin xyz="0 0 0" rpy="0 0 0"/>
+      		<mass value="0.5"/>
+      		<inertia
+        		ixx="1.0" ixy="0.0" ixz="0.0"
+        		iyy="1.0" iyz="0.0"
+        		izz="1.0"/>
+    	</inertial>
 	</link>
     <link name="elbow_link">
@@ -113,4 +146,12 @@
             </geometry>
         </collision>
+		<inertial>
+      		<origin xyz="0 0 0" rpy="0 0 0"/>
+      		<mass value="0.4"/>
+      		<inertia
+        		ixx="1.0" ixy="0.0" ixz="0.0"
+        		iyy="1.0" iyz="0.0"
+        		izz="1.0"/>
+    	</inertial>
 	</link>
     <link name="forearm_link">
@@ -130,4 +171,12 @@
             </geometry>
         </collision>
+		<inertial>
+      		<origin xyz="0 0 0" rpy="0 0 0"/>
+      		<mass value="0.3"/>
+      		<inertia
+        		ixx="1.0" ixy="0.0" ixz="0.0"
+        		iyy="1.0" iyz="0.0"
+        		izz="1.0"/>
+    	</inertial>
 	</link>
     <link name="wrist_link">
@@ -147,4 +196,12 @@
             </geometry>
         </collision>
+		<inertial>
+      		<origin xyz="0 0 0" rpy="0 0 0"/>
+      		<mass value="0.2"/>
+      		<inertia
+        		ixx="1.0" ixy="0.0" ixz="0.0"
+        		iyy="1.0" iyz="0.0"
+        		izz="1.0"/>
+    	</inertial>
 	</link>
     <link name="hand_link">
@@ -164,4 +221,12 @@
             </geometry>
         </collision>
+		<inertial>
+      		<origin xyz="0 0 0" rpy="0 0 0"/>
+      		<mass value="0.1"/>
+      		<inertia
+        		ixx="1.0" ixy="0.0" ixz="0.0"
+        		iyy="1.0" iyz="0.0"
+        		izz="1.0"/>
+    	</inertial>
 	</link>
     <link name="gripper_link">
