Commit message: change color tag

File: niryo_one_description/urdf/v1/niryo_one.gazebo.xacro (robot description, xacro)
@@ -1,37 +1,52 @@
 <?xml version="1.0"?>
 <robot xmlns:xacro="http://www.ros.org/wiki/xacro" name="niryo_one">
-    <gazebo reference="ground_link">
+  <gazebo reference="ground_link">
+		<material>Gazebo/Blue</material>
 		<turnGravityOff>true</turnGravityOff>
 	</gazebo>
   <gazebo reference="base_link">
-		<material>>Gazebo/Blue</material>
+		<material>>Gazebo/Black</material>
 		<turnGravityOff>true</turnGravityOff>
 	</gazebo>
-    <gazebo reference="shoulder_link">
+  <gazebo reference="shoulder_link">
 		<material>Gazebo/Black</material>
+		  <mu1>0.0</mu1>
+  		<mu2>0.0</mu2>
 		<turnGravityOff>true</turnGravityOff>
 	</gazebo>
-    <gazebo reference="arm_link">
+  <gazebo reference="arm_link">
 		<material>Gazebo/Blue</material>
+		<mu1>0.0</mu1>
+  	<mu2>0.0</mu2>
 		<turnGravityOff>true</turnGravityOff>
 	</gazebo>
-    <gazebo reference="elbow_link">
+  <gazebo reference="elbow_link">
 		<material>Gazebo/Black</material>
+		<mu1>0.0</mu1>
+  	<mu2>0.0</mu2>
 		<turnGravityOff>true</turnGravityOff>
 	</gazebo>
-    <gazebo reference="forearm_link">
+  <gazebo reference="forearm_link">
 		<material>Gazebo/Blue</material>
+		<mu1>0.0</mu1>
+  	<mu2>0.0</mu2>
 		<turnGravityOff>true</turnGravityOff>
 	</gazebo>
   <gazebo reference="wrist_link">
 		<material>Gazebo/Black</material>
+		<mu1>0.0</mu1>
+  	<mu2>0.0</mu2>
 		<turnGravityOff>true</turnGravityOff>
 	</gazebo>
   <gazebo reference="hand_link">
 		<material>Gazebo/Blue</material>
+		<mu1>0.0</mu1>
+  	<mu2>0.0</mu2>
 		<turnGravityOff>true</turnGravityOff>
 	</gazebo>
 	<gazebo reference="gripper_link">
 		<material>Gazebo/Black</material>
+		<mu1>0.0</mu1>
+  	<mu2>0.0</mu2>
 		<turnGravityOff>true</turnGravityOff>
 	</gazebo>
