Commit message: add transmission tag for robot control

File: niryo_one_description/urdf/v1/niryo_one.urdf.xacro (robot description, xacro)
@@ -46,7 +46,23 @@
 	<!-- Links -->
     <link name="ground_link"/>
-		<inertial>
-			<origin xyz="0 0 0" rpy="0 0 0"/>
-      		<mass value="1"/>
+    <link name="base_link">
+		<visual>
+			<origin xyz="0 0 0" rpy="0 0 0" />
+			<geometry>
+                <mesh filename="package://niryo_one_description/meshes/collada/base_link.dae" />
+			</geometry>
+			<material name="">
+				<color rgba="0.2 0.6 1 1" />
+			</material>
+        </visual>
+        <collision>
+			<origin xyz="0 0 0" rpy="0 0 0" />
+            <geometry>
+                <mesh filename="package://niryo_one_description/meshes/stl/base_link.stl" />
+            </geometry>
+        </collision>
+		<inertial>
+      		<origin xyz="0 0 0" rpy="0 0 0"/>
+      		<mass value="1.3"/>
       		<inertia
         		ixx="0.0" ixy="0.0" ixz="0.0"
@@ -54,63 +70,39 @@
         		izz="0.0"/>
     	</inertial>
-    <link name="base_link">
-		<visual>
-			<origin xyz="0 0 0" rpy="0 0 0" />
-			<geometry>
-                <mesh filename="package://niryo_one_description/meshes/collada/base_link.dae" />
+	</link>
+    <link name="shoulder_link">
+		<visual>
+			<origin xyz="0 0 0" rpy="0 0 0" />
+			<geometry>
+                <mesh filename="package://niryo_one_description/meshes/collada/shoulder_link.dae" />
+			</geometry>
+			<material name="">
+				<color rgba="0.8 0.8 0.8 1" />
+			</material>
+		</visual>
+        <collision>
+			<origin xyz="0 0 0" rpy="0 0 0" />
+            <geometry>
+                <mesh filename="package://niryo_one_description/meshes/stl/shoulder_link.stl" />
+            </geometry>
+        </collision>
+		<inertial>
+      		<origin xyz="0 0 0" rpy="0 0 0"/>
+      		<mass value="0.6"/>
+      		<inertia
+        		ixx="1.0" ixy="0.0" ixz="0.0"
+        		iyy="1.0" iyz="0.0"
+        		izz="1.0"/>
+    	</inertial>
+	</link>
+    <link name="arm_link">
+		<visual>
+			<origin xyz="0 0 0" rpy="0 0 0" />
+			<geometry>
+                <mesh filename="package://niryo_one_description/meshes/collada/arm_link.dae" />
 			</geometry>
 			<material name="">
 				<color rgba="0.2 0.6 1 1" />
 			</material>
-        </visual>
-        <collision>
-			<origin xyz="0 0 0" rpy="0 0 0" />
-            <geometry>
-                <mesh filename="package://niryo_one_description/meshes/stl/base_link.stl" />
-            </geometry>
-        </collision>
-		<inertial>
-      		<origin xyz="0 0 0" rpy="0 0 0"/>
-      		<mass value="1.3"/>
-      		<inertia
-        		ixx="0.0" ixy="0.0" ixz="0.0"
-        		iyy="0.0" iyz="0.0"
-        		izz="0.0"/>
-    	</inertial>
-	</link>
-    <link name="shoulder_link">
-		<visual>
-			<origin xyz="0 0 0" rpy="0 0 0" />
-			<geometry>
-                <mesh filename="package://niryo_one_description/meshes/collada/shoulder_link.dae" />
-			</geometry>
-			<material name="">
-				<color rgba="0.8 0.8 0.8 1" />
-			</material>
-		</visual>
-        <collision>
-			<origin xyz="0 0 0" rpy="0 0 0" />
-            <geometry>
-                <mesh filename="package://niryo_one_description/meshes/stl/shoulder_link.stl" />
-            </geometry>
-        </collision>
-		<inertial>
-      		<origin xyz="0 0 0" rpy="0 0 0"/>
-      		<mass value="0.6"/>
-      		<inertia
-        		ixx="1.0" ixy="0.0" ixz="0.0"
-        		iyy="1.0" iyz="0.0"
-        		izz="1.0"/>
-    	</inertial>
-	</link>
-    <link name="arm_link">
-		<visual>
-			<origin xyz="0 0 0" rpy="0 0 0" />
-			<geometry>
-                <mesh filename="package://niryo_one_description/meshes/collada/arm_link.dae" />
-			</geometry>
-			<material name="">
-				<color rgba="0.2 0.6 1 1" />
-			</material>
 		</visual>
         <collision>
@@ -133,5 +125,5 @@
 			<origin xyz="0 0 0" rpy="0 0 0" />
 			<geometry>
-                <!--	<box size="0.1 0.1 0.048"/> -->
+            	<!--box size="0.01 0.01 0.01"/-->
                 <mesh filename="package://niryo_one_description/meshes/collada/elbow_link.dae" />
 			</geometry>
@@ -285,3 +277,66 @@
         <origin xyz="0 0 ${distance_hand_gripper}" rpy="${-PI/2} ${-PI/2} 0" />
 	</joint>
+	<!--transmission-->
+	<transmission name="base_shoulder_transmission">
+      <type>transmission_interface/SimpleTransmission</type>
+      <joint name="joint_1">
+        <hardwareInterface>hardware_interface/PositionJointInterface</hardwareInterface>
+      </joint>
+      <actuator name="base_shoulder_motor">
+        <mechanicalReduction>1</mechanicalReduction>
+		<hardwareInterface>hardware_interface/PositionJointInterface</hardwareInterface>
+      </actuator>
+    </transmission>
+	<transmission name="shoulder_arm_transmission">
+      <type>transmission_interface/SimpleTransmission</type>
+      <joint name="joint_2">
+        <hardwareInterface>hardware_interface/PositionJointInterface</hardwareInterface>
+      </joint>
+      <actuator name="shoulder_arm_motor">
+        <mechanicalReduction>1</mechanicalReduction>
+		<hardwareInterface>hardware_interface/PositionJointInterface</hardwareInterface>
+      </actuator>
+    </transmission>
+	<transmission name="arm_elbow_transmission">
+      <type>transmission_interface/SimpleTransmission</type>
+      <joint name="joint_3">
+        <hardwareInterface>hardware_interface/PositionJointInterface</hardwareInterface>
+      </joint>
+      <actuator name="arm_elbow_motor">
+        <mechanicalReduction>1</mechanicalReduction>
+		<hardwareInterface>hardware_interface/PositionJointInterface</hardwareInterface>
+      </actuator>
+    </transmission>
+	<transmission name="elbow_forarm_transmission">
+      <type>transmission_interface/SimpleTransmission</type>
+      <joint name="joint_4">
+        <hardwareInterface>hardware_interface/PositionJointInterface</hardwareInterface>
+      </joint>
+      <actuator name="elbow_forarm_motor">
+        <mechanicalReduction>1</mechanicalReduction>
+      </actuator>
+    </transmission>
+	<transmission name="forarm_wirst_transmission">
+      <type>transmission_interface/SimpleTransmission</type>
+      <joint name="joint_5">
+        <hardwareInterface>hardware_interface/PositionJointInterface</hardwareInterface>
+      </joint>
+      <actuator name="forarm_wirst_motor">
+        <mechanicalReduction>1</mechanicalReduction>
+      </actuator>
+    </transmission>
+	<transmission name="wirst_gripper_transmission">
+      <type>transmission_interface/SimpleTransmission</type>
+      <joint name="joint_6">
+        <hardwareInterface>hardware_interface/PositionJointInterface</hardwareInterface>
+      </joint>
+      <actuator name="wirst_gripper_motor">
+        <mechanicalReduction>1</mechanicalReduction>
+      </actuator>
+    </transmission>
+	<!--plugin-->
+	<gazebo>
+  		<plugin name="gazebo_ros_control" filename="libgazebo_ros_control.so">
+  		</plugin>
+  	</gazebo>
 </robot>

Commit message: Update URDF with hw V2.0 values

File: niryo_one_description/urdf/v1/niryo_one.urdf.xacro (robot description, xacro)
@@ -26,6 +26,5 @@
     <xacro:property name="distance_wrist_hand_x" value="0.018" />
     <xacro:property name="distance_wrist_hand_y" value="0" />
-    <!-- not yet implemented, for now -->
-    <xacro:property name="distance_hand_gripper" value="0.00" />
+    <xacro:property name="distance_hand_tool" value="0.00" />
 	<xacro:property name="thickness_arm_axis" value="0.052" />
 	<xacro:property name="thickness_forearm_axis" value="0.048" />
@@ -165,5 +164,5 @@
         </collision>
 	</link>
-    <link name="gripper_link">
+    <link name="tool_link">
 	</link>
 	<!--Joints -->
@@ -215,8 +214,8 @@
 		<axis xyz="0 0 1" />
 	</joint>
-	<joint name="hand_gripper_joint" type="fixed">
+	<joint name="hand_tool_joint" type="fixed">
         <parent link="hand_link" />
-        <child link="gripper_link" />
-        <origin xyz="0 0 ${distance_hand_gripper}" rpy="${-PI/2} ${-PI/2} 0" />
+        <child link="tool_link" />
+        <origin xyz="0 0 ${distance_hand_tool}" rpy="${-PI/2} ${-PI/2} 0" />
 	</joint>
 </robot>

File: niryo_one_description/urdf/v1/without_mesh_niryo_one.urdf.xacro (robot description, xacro)
@@ -26,6 +26,5 @@
 	<xacro:property name="distance_wrist_hand_x" value="0.018" />
     <xacro:property name="distance_wrist_hand_y" value="0" />
-    <!-- not yet implemented, tools are handled separately -->
-    <xacro:property name="distance_hand_gripper" value="0.00" />
+    <xacro:property name="distance_hand_tool" value="0.00" />
 	<xacro:property name="thickness_arm_axis" value="0.052" />
 	<xacro:property name="thickness_forearm_axis" value="0.048" />
@@ -59,5 +58,5 @@
     <link name="hand_link">
 	</link>
-    <link name="gripper_link">
+    <link name="tool_link">
 	</link>
 	<!--Joints -->
@@ -109,8 +108,8 @@
 		<axis xyz="0 0 1" />
 	</joint>
-	<joint name="hand_gripper_joint" type="fixed">
+	<joint name="hand_tool_joint" type="fixed">
         <parent link="hand_link" />
-        <child link="gripper_link" />
-        <origin xyz="0 0 ${distance_hand_gripper}" rpy="${-PI/2} ${-PI/2} 0" />
+        <child link="tool_link" />
+        <origin xyz="0 0 ${distance_hand_tool}" rpy="${-PI/2} ${-PI/2} 0" />
 	</joint>
 </robot>

File: niryo_one_description/urdf/v2/niryo_one.urdf.xacro (robot description, xacro)
@@ -1,6 +1,4 @@
 <?xml version="1.0"?>
 <!--
-    Work in progress
-    Will be updated with hw V2 values
     niryo_one.urdf.xacro
     Copyright (C) 2017 Niryo
@@ -20,14 +18,13 @@
 	<!-- Properties -->
     <xacro:property name="distance_origin_shoulder_z" value="0.103" />
-    <xacro:property name="distance_shoulder_arm_z" value="0.08" />
-    <xacro:property name="distance_arm_elbow_x" value="0.21004" />
+    <xacro:property name="distance_shoulder_arm_z" value="0.080" />
+    <xacro:property name="distance_arm_elbow_x" value="0.209" />
     <xacro:property name="distance_arm_elbow_y" value="0.0" />
-    <xacro:property name="distance_elbow_forearm_x" value="0.037" />
-    <xacro:property name="distance_elbow_forearm_y" value="0.032" />
-    <xacro:property name="distance_forearm_wrist_z" value="0.180" />
-    <xacro:property name="distance_wrist_hand_x" value="0.018" />
-    <xacro:property name="distance_wrist_hand_y" value="0" />
-    <!-- not yet implemented, for now -->
-    <xacro:property name="distance_hand_gripper" value="0.00" />
+    <xacro:property name="distance_elbow_forearm_x" value="0.042" />
+    <xacro:property name="distance_elbow_forearm_y" value="0.030" />
+    <xacro:property name="distance_forearm_wrist_z" value="0.179" />
+    <xacro:property name="distance_wrist_hand_x" value="0.0164" />
+    <xacro:property name="distance_wrist_hand_y" value="-0.0055" />
+    <xacro:property name="distance_hand_tool" value="0.00" />
 	<xacro:property name="thickness_arm_axis" value="0.052" />
 	<xacro:property name="thickness_forearm_axis" value="0.048" />
@@ -53,7 +50,4 @@
                 <mesh filename="package://niryo_one_description/meshes/collada/base_link.dae" />
 			</geometry>
-			<material name="">
-				<color rgba="0.2 0.6 1 1" />
-			</material>
         </visual>
         <collision>
@@ -70,7 +64,4 @@
                 <mesh filename="package://niryo_one_description/meshes/collada/shoulder_link.dae" />
 			</geometry>
-			<material name="">
-				<color rgba="0.8 0.8 0.8 1" />
-			</material>
 		</visual>
         <collision>
@@ -87,7 +78,4 @@
                 <mesh filename="package://niryo_one_description/meshes/collada/arm_link.dae" />
 			</geometry>
-			<material name="">
-				<color rgba="0.2 0.6 1 1" />
-			</material>
 		</visual>
         <collision>
@@ -102,10 +90,6 @@
 			<origin xyz="0 0 0" rpy="0 0 0" />
 			<geometry>
-                <!--	<box size="0.1 0.1 0.048"/> -->
                 <mesh filename="package://niryo_one_description/meshes/collada/elbow_link.dae" />
 			</geometry>
-			<material name="">
-				<color rgba="0.8 0.8 0.8 1" />
-			</material>
 		</visual>
         <collision>
@@ -122,7 +106,4 @@
                 <mesh filename="package://niryo_one_description/meshes/collada/forearm_link.dae" />
 			</geometry>
-			<material name="">
-				<color rgba="0.2 0.6 1 1" />
-			</material>
 		</visual>
         <collision>
@@ -139,7 +120,4 @@
                 <mesh filename="package://niryo_one_description/meshes/collada/wrist_link.dae" />
 			</geometry>
-			<material name="">
-				<color rgba="0.8 0.8 0.8 1" />
-			</material>
 		</visual>
         <collision>
@@ -156,7 +134,4 @@
                 <mesh filename="package://niryo_one_description/meshes/collada/hand_link.dae" />
 			</geometry>
-			<material name="">
-				<color rgba="0.6 0 0 1" />
-			</material>
 		</visual>
         <collision>
@@ -167,5 +142,5 @@
         </collision>
 	</link>
-    <link name="gripper_link">
+    <link name="tool_link">
 	</link>
 	<!--Joints -->
@@ -217,8 +192,8 @@
 		<axis xyz="0 0 1" />
 	</joint>
-	<joint name="hand_gripper_joint" type="fixed">
+	<joint name="hand_tool_joint" type="fixed">
         <parent link="hand_link" />
-        <child link="gripper_link" />
-        <origin xyz="0 0 ${distance_hand_gripper}" rpy="${-PI/2} ${-PI/2} 0" />
+        <child link="tool_link" />
+        <origin xyz="0 0 ${distance_hand_tool}" rpy="${-PI/2} ${-PI/2} 0" />
 	</joint>
 </robot>

File: niryo_one_description/urdf/v2/without_mesh_niryo_one.urdf.xacro (robot description, xacro)
@@ -1,6 +1,4 @@
 <?xml version="1.0"?>
 <!--
-    Work in progress
-    Will be updated with hw V2 values
     without_mesh_niryo_one.urdf.xacro
     Copyright (C) 2017 Niryo
@@ -19,15 +17,14 @@
 <robot xmlns:xacro="http://www.ros.org/wiki/xacro" name="niryo_one">
 	<!-- Properties -->
-	<xacro:property name="distance_origin_shoulder_z" value="0.103" />
-	<xacro:property name="distance_shoulder_arm_z" value="0.08" />
-    <xacro:property name="distance_arm_elbow_x" value="0.21004" />
+    <xacro:property name="distance_origin_shoulder_z" value="0.103" />
+    <xacro:property name="distance_shoulder_arm_z" value="0.080" />
+    <xacro:property name="distance_arm_elbow_x" value="0.209" />
     <xacro:property name="distance_arm_elbow_y" value="0.0" />
-    <xacro:property name="distance_elbow_forearm_x" value="0.037" />
-    <xacro:property name="distance_elbow_forearm_y" value="0.032" />
-    <xacro:property name="distance_forearm_wrist_z" value="0.180" />
-	<xacro:property name="distance_wrist_hand_x" value="0.018" />
-    <xacro:property name="distance_wrist_hand_y" value="0" />
-    <!-- not yet implemented, tools are handled separately -->
-    <xacro:property name="distance_hand_gripper" value="0.00" />
+    <xacro:property name="distance_elbow_forearm_x" value="0.042" />
+    <xacro:property name="distance_elbow_forearm_y" value="0.030" />
+    <xacro:property name="distance_forearm_wrist_z" value="0.179" />
+    <xacro:property name="distance_wrist_hand_x" value="0.0164" />
+    <xacro:property name="distance_wrist_hand_y" value="-0.0055" />
+    <xacro:property name="distance_hand_tool" value="0.00" />
 	<xacro:property name="thickness_arm_axis" value="0.052" />
 	<xacro:property name="thickness_forearm_axis" value="0.048" />
@@ -61,5 +58,5 @@
     <link name="hand_link">
 	</link>
-    <link name="gripper_link">
+    <link name="tool_link">
 	</link>
 	<!--Joints -->
@@ -111,8 +108,8 @@
 		<axis xyz="0 0 1" />
 	</joint>
-	<joint name="hand_gripper_joint" type="fixed">
+	<joint name="hand_tool_joint" type="fixed">
         <parent link="hand_link" />
-        <child link="gripper_link" />
-        <origin xyz="0 0 ${distance_hand_gripper}" rpy="${-PI/2} ${-PI/2} 0" />
+        <child link="tool_link" />
+        <origin xyz="0 0 ${distance_hand_tool}" rpy="${-PI/2} ${-PI/2} 0" />
 	</joint>
 </robot>
