Commit message: Add stl, collada files for hw V2.0 and update urdf, srdf, config files

File: niryo_one_description/urdf/v1/niryo_one.urdf.xacro (robot description, xacro)
@@ -27,6 +27,4 @@
     <xacro:property name="distance_wrist_hand_y" value="0" />
     <xacro:property name="distance_hand_tool" value="0.00" />
-	<xacro:property name="thickness_arm_axis" value="0.052" />
-	<xacro:property name="thickness_forearm_axis" value="0.048" />
 	<xacro:property name="PI" value="3.14159265359" />
     <xacro:property name="limit_low_shoulder_rotation" value="-3.05433" />
@@ -48,5 +46,5 @@
 			<origin xyz="0 0 0" rpy="0 0 0" />
 			<geometry>
-                <mesh filename="package://niryo_one_description/meshes/collada/base_link.dae" />
+                <mesh filename="package://niryo_one_description/meshes/v1/collada/base_link.dae" />
 			</geometry>
 			<material name="">
@@ -57,5 +55,5 @@
 			<origin xyz="0 0 0" rpy="0 0 0" />
             <geometry>
-                <mesh filename="package://niryo_one_description/meshes/stl/base_link.stl" />
+                <mesh filename="package://niryo_one_description/meshes/v1/stl/base_link.stl" />
             </geometry>
         </collision>
@@ -65,5 +63,5 @@
 			<origin xyz="0 0 0" rpy="0 0 0" />
 			<geometry>
-                <mesh filename="package://niryo_one_description/meshes/collada/shoulder_link.dae" />
+                <mesh filename="package://niryo_one_description/meshes/v1/collada/shoulder_link.dae" />
 			</geometry>
 			<material name="">
@@ -74,5 +72,5 @@
 			<origin xyz="0 0 0" rpy="0 0 0" />
             <geometry>
-                <mesh filename="package://niryo_one_description/meshes/stl/shoulder_link.stl" />
+                <mesh filename="package://niryo_one_description/meshes/v1/stl/shoulder_link.stl" />
             </geometry>
         </collision>
@@ -82,5 +80,5 @@
 			<origin xyz="0 0 0" rpy="0 0 0" />
 			<geometry>
-                <mesh filename="package://niryo_one_description/meshes/collada/arm_link.dae" />
+                <mesh filename="package://niryo_one_description/meshes/v1/collada/arm_link.dae" />
 			</geometry>
 			<material name="">
@@ -91,5 +89,5 @@
 			<origin xyz="0 0 0" rpy="0 0 0" />
             <geometry>
-                <mesh filename="package://niryo_one_description/meshes/stl/arm_link.stl" />
+                <mesh filename="package://niryo_one_description/meshes/v1/stl/arm_link.stl" />
             </geometry>
         </collision>
@@ -100,5 +98,5 @@
 			<geometry>
                 <!--	<box size="0.1 0.1 0.048"/> -->
-                <mesh filename="package://niryo_one_description/meshes/collada/elbow_link.dae" />
+                <mesh filename="package://niryo_one_description/meshes/v1/collada/elbow_link.dae" />
 			</geometry>
 			<material name="">
@@ -109,5 +107,5 @@
 			<origin xyz="0 0 0" rpy="0 0 0" />
             <geometry>
-                <mesh filename="package://niryo_one_description/meshes/stl/elbow_link.stl" />
+                <mesh filename="package://niryo_one_description/meshes/v1/stl/elbow_link.stl" />
             </geometry>
         </collision>
@@ -117,5 +115,5 @@
 			<origin xyz="0 0 0" rpy="0 0 0" />
 			<geometry>
-                <mesh filename="package://niryo_one_description/meshes/collada/forearm_link.dae" />
+                <mesh filename="package://niryo_one_description/meshes/v1/collada/forearm_link.dae" />
 			</geometry>
 			<material name="">
@@ -126,5 +124,5 @@
 			<origin xyz="0 0 0" rpy="0 0 0" />
             <geometry>
-                <mesh filename="package://niryo_one_description/meshes/stl/forearm_link.stl" />
+                <mesh filename="package://niryo_one_description/meshes/v1/stl/forearm_link.stl" />
             </geometry>
         </collision>
@@ -134,5 +132,5 @@
 			<origin xyz="0 0 0" rpy="0 0 0" />
 			<geometry>
-                <mesh filename="package://niryo_one_description/meshes/collada/wrist_link.dae" />
+                <mesh filename="package://niryo_one_description/meshes/v1/collada/wrist_link.dae" />
 			</geometry>
 			<material name="">
@@ -143,5 +141,5 @@
 			<origin xyz="0 0 0" rpy="0 0 0" />
             <geometry>
-                <mesh filename="package://niryo_one_description/meshes/stl/wrist_link.stl" />
+                <mesh filename="package://niryo_one_description/meshes/v1/stl/wrist_link.stl" />
             </geometry>
         </collision>
@@ -151,5 +149,5 @@
 			<origin xyz="0 0 0" rpy="0 0 0" />
 			<geometry>
-                <mesh filename="package://niryo_one_description/meshes/collada/hand_link.dae" />
+                <mesh filename="package://niryo_one_description/meshes/v1/collada/hand_link.dae" />
 			</geometry>
 			<material name="">
@@ -160,5 +158,5 @@
 			<origin xyz="0 0 0" rpy="0 0 0" />
             <geometry>
-                <mesh filename="package://niryo_one_description/meshes/stl/hand_link.stl" />
+                <mesh filename="package://niryo_one_description/meshes/v1/stl/hand_link.stl" />
             </geometry>
         </collision>

File: niryo_one_description/urdf/v1/without_mesh_niryo_one.urdf.xacro (robot description, xacro)
@@ -27,6 +27,4 @@
     <xacro:property name="distance_wrist_hand_y" value="0" />
     <xacro:property name="distance_hand_tool" value="0.00" />
-	<xacro:property name="thickness_arm_axis" value="0.052" />
-	<xacro:property name="thickness_forearm_axis" value="0.048" />
 	<xacro:property name="PI" value="3.14159265359" />
 	<xacro:property name="limit_low_shoulder_rotation" value="-3.05433" />

File: niryo_one_description/urdf/v2/niryo_one.urdf.xacro (robot description, xacro)
@@ -19,27 +19,25 @@
     <xacro:property name="distance_origin_shoulder_z" value="0.103" />
     <xacro:property name="distance_shoulder_arm_z" value="0.080" />
-    <xacro:property name="distance_arm_elbow_x" value="0.209" />
+    <xacro:property name="distance_arm_elbow_x" value="0.210" />
     <xacro:property name="distance_arm_elbow_y" value="0.0" />
-    <xacro:property name="distance_elbow_forearm_x" value="0.042" />
+    <xacro:property name="distance_elbow_forearm_x" value="0.0415" />
     <xacro:property name="distance_elbow_forearm_y" value="0.030" />
-    <xacro:property name="distance_forearm_wrist_z" value="0.179" />
+    <xacro:property name="distance_forearm_wrist_z" value="0.180" />
     <xacro:property name="distance_wrist_hand_x" value="0.0164" />
     <xacro:property name="distance_wrist_hand_y" value="-0.0055" />
-    <xacro:property name="distance_hand_tool" value="0.00" />
-	<xacro:property name="thickness_arm_axis" value="0.052" />
-	<xacro:property name="thickness_forearm_axis" value="0.048" />
+    <xacro:property name="distance_hand_tool" value="0.0073" />
 	<xacro:property name="PI" value="3.14159265359" />
     <xacro:property name="limit_low_shoulder_rotation" value="-3.05433" />
     <xacro:property name="limit_up_shoulder_rotation" value="3.05433" />
-    <xacro:property name="limit_low_arm_rotation" value="${-PI/2}" />
-    <xacro:property name="limit_up_arm_rotation" value="0.628319" />
-    <xacro:property name="limit_low_elbow_rotation" value="-1.401" />
-    <xacro:property name="limit_up_elbow_rotation" value="0.994838" />
-    <xacro:property name="limit_low_forearm_rotation" value="-2.61799" />
-    <xacro:property name="limit_up_forearm_rotation" value="2.61799" />
-    <xacro:property name="limit_low_wrist_rotation" value="-2.26893" />
-    <xacro:property name="limit_up_wrist_rotation" value="2.26893" />
-    <xacro:property name="limit_low_hand_rotation" value="-2.57" />
-    <xacro:property name="limit_up_hand_rotation" value="2.57" />
+    <xacro:property name="limit_low_arm_rotation" value="-1.91986" />
+    <xacro:property name="limit_up_arm_rotation" value="0.640187" />
+    <xacro:property name="limit_low_elbow_rotation" value="-1.397485" />
+    <xacro:property name="limit_up_elbow_rotation" value="${PI/2}" />
+    <xacro:property name="limit_low_forearm_rotation" value="-3.05433" />
+    <xacro:property name="limit_up_forearm_rotation" value="3.05433" />
+    <xacro:property name="limit_low_wrist_rotation" value="-2.0944" />
+    <xacro:property name="limit_up_wrist_rotation" value="2.53073" />
+    <xacro:property name="limit_low_hand_rotation" value="-2.57436" />
+    <xacro:property name="limit_up_hand_rotation" value="2.57436" />
 	<!-- Links -->
     <link name="ground_link"/>
@@ -48,5 +46,5 @@
 			<origin xyz="0 0 0" rpy="0 0 0" />
 			<geometry>
-                <mesh filename="package://niryo_one_description/meshes/collada/base_link.dae" />
+                <mesh filename="package://niryo_one_description/meshes/v2/collada/base_link.dae" />
 			</geometry>
         </visual>
@@ -54,5 +52,5 @@
 			<origin xyz="0 0 0" rpy="0 0 0" />
             <geometry>
-                <mesh filename="package://niryo_one_description/meshes/stl/base_link.stl" />
+                <mesh filename="package://niryo_one_description/meshes/v2/stl/base_link.stl" />
             </geometry>
         </collision>
@@ -62,5 +60,5 @@
 			<origin xyz="0 0 0" rpy="0 0 0" />
 			<geometry>
-                <mesh filename="package://niryo_one_description/meshes/collada/shoulder_link.dae" />
+                <mesh filename="package://niryo_one_description/meshes/v2/collada/shoulder_link.dae" />
 			</geometry>
 		</visual>
@@ -68,5 +66,5 @@
 			<origin xyz="0 0 0" rpy="0 0 0" />
             <geometry>
-                <mesh filename="package://niryo_one_description/meshes/stl/shoulder_link.stl" />
+                <mesh filename="package://niryo_one_description/meshes/v2/stl/shoulder_link.stl" />
             </geometry>
         </collision>
@@ -76,5 +74,5 @@
 			<origin xyz="0 0 0" rpy="0 0 0" />
 			<geometry>
-                <mesh filename="package://niryo_one_description/meshes/collada/arm_link.dae" />
+                <mesh filename="package://niryo_one_description/meshes/v2/collada/arm_link.dae" />
 			</geometry>
 		</visual>
@@ -82,5 +80,5 @@
 			<origin xyz="0 0 0" rpy="0 0 0" />
             <geometry>
-                <mesh filename="package://niryo_one_description/meshes/stl/arm_link.stl" />
+                <mesh filename="package://niryo_one_description/meshes/v2/stl/arm_link.stl" />
             </geometry>
         </collision>
@@ -90,5 +88,5 @@
 			<origin xyz="0 0 0" rpy="0 0 0" />
 			<geometry>
-                <mesh filename="package://niryo_one_description/meshes/collada/elbow_link.dae" />
+                <mesh filename="package://niryo_one_description/meshes/v2/collada/elbow_link.dae" />
 			</geometry>
 		</visual>
@@ -96,5 +94,5 @@
 			<origin xyz="0 0 0" rpy="0 0 0" />
             <geometry>
-                <mesh filename="package://niryo_one_description/meshes/stl/elbow_link.stl" />
+                <mesh filename="package://niryo_one_description/meshes/v2/stl/elbow_link.stl" />
             </geometry>
         </collision>
@@ -104,5 +102,5 @@
 			<origin xyz="0 0 0" rpy="0 0 0" />
 			<geometry>
-                <mesh filename="package://niryo_one_description/meshes/collada/forearm_link.dae" />
+                <mesh filename="package://niryo_one_description/meshes/v2/collada/forearm_link.dae" />
 			</geometry>
 		</visual>
@@ -110,5 +108,5 @@
 			<origin xyz="0 0 0" rpy="0 0 0" />
             <geometry>
-                <mesh filename="package://niryo_one_description/meshes/stl/forearm_link.stl" />
+                <mesh filename="package://niryo_one_description/meshes/v2/stl/forearm_link.stl" />
             </geometry>
         </collision>
@@ -118,5 +116,5 @@
 			<origin xyz="0 0 0" rpy="0 0 0" />
 			<geometry>
-                <mesh filename="package://niryo_one_description/meshes/collada/wrist_link.dae" />
+                <mesh filename="package://niryo_one_description/meshes/v2/collada/wrist_link.dae" />
 			</geometry>
 		</visual>
@@ -124,5 +122,5 @@
 			<origin xyz="0 0 0" rpy="0 0 0" />
             <geometry>
-                <mesh filename="package://niryo_one_description/meshes/stl/wrist_link.stl" />
+                <mesh filename="package://niryo_one_description/meshes/v2/stl/wrist_link.stl" />
             </geometry>
         </collision>
@@ -132,5 +130,5 @@
 			<origin xyz="0 0 0" rpy="0 0 0" />
 			<geometry>
-                <mesh filename="package://niryo_one_description/meshes/collada/hand_link.dae" />
+                <mesh filename="package://niryo_one_description/meshes/v2/collada/hand_link.dae" />
 			</geometry>
 		</visual>
@@ -138,5 +136,5 @@
 			<origin xyz="0 0 0" rpy="0 0 0" />
             <geometry>
-                <mesh filename="package://niryo_one_description/meshes/stl/hand_link.stl" />
+                <mesh filename="package://niryo_one_description/meshes/v2/stl/hand_link.stl" />
             </geometry>
         </collision>

File: niryo_one_description/urdf/v2/without_mesh_niryo_one.urdf.xacro (robot description, xacro)
@@ -19,27 +19,25 @@
     <xacro:property name="distance_origin_shoulder_z" value="0.103" />
     <xacro:property name="distance_shoulder_arm_z" value="0.080" />
-    <xacro:property name="distance_arm_elbow_x" value="0.209" />
+    <xacro:property name="distance_arm_elbow_x" value="0.210" />
     <xacro:property name="distance_arm_elbow_y" value="0.0" />
-    <xacro:property name="distance_elbow_forearm_x" value="0.042" />
+    <xacro:property name="distance_elbow_forearm_x" value="0.0415" />
     <xacro:property name="distance_elbow_forearm_y" value="0.030" />
-    <xacro:property name="distance_forearm_wrist_z" value="0.179" />
+    <xacro:property name="distance_forearm_wrist_z" value="0.180" />
     <xacro:property name="distance_wrist_hand_x" value="0.0164" />
     <xacro:property name="distance_wrist_hand_y" value="-0.0055" />
-    <xacro:property name="distance_hand_tool" value="0.00" />
-	<xacro:property name="thickness_arm_axis" value="0.052" />
-	<xacro:property name="thickness_forearm_axis" value="0.048" />
+    <xacro:property name="distance_hand_tool" value="0.0073" />
 	<xacro:property name="PI" value="3.14159265359" />
-	<xacro:property name="limit_low_shoulder_rotation" value="-3.05433" />
-	<xacro:property name="limit_up_shoulder_rotation" value="3.05433" />
-    <xacro:property name="limit_low_arm_rotation" value="${-PI/2}" />
-    <xacro:property name="limit_up_arm_rotation" value="0.628319" />
-    <xacro:property name="limit_low_elbow_rotation" value="-1.401" />
-    <xacro:property name="limit_up_elbow_rotation" value="0.994838" />
-    <xacro:property name="limit_low_forearm_rotation" value="-2.61799" />
-    <xacro:property name="limit_up_forearm_rotation" value="2.61799" />
-    <xacro:property name="limit_low_wrist_rotation" value="-2.26893" />
-    <xacro:property name="limit_up_wrist_rotation" value="2.26893" />
-    <xacro:property name="limit_low_hand_rotation" value="-2.57" />
-    <xacro:property name="limit_up_hand_rotation" value="2.57" />
+    <xacro:property name="limit_low_shoulder_rotation" value="-3.05433" />
+    <xacro:property name="limit_up_shoulder_rotation" value="3.05433" />
+    <xacro:property name="limit_low_arm_rotation" value="-1.91986" />
+    <xacro:property name="limit_up_arm_rotation" value="0.640187" />
+    <xacro:property name="limit_low_elbow_rotation" value="-1.397485" />
+    <xacro:property name="limit_up_elbow_rotation" value="${PI/2}" />
+    <xacro:property name="limit_low_forearm_rotation" value="-3.05433" />
+    <xacro:property name="limit_up_forearm_rotation" value="3.05433" />
+    <xacro:property name="limit_low_wrist_rotation" value="-2.0944" />
+    <xacro:property name="limit_up_wrist_rotation" value="2.53073" />
+    <xacro:property name="limit_low_hand_rotation" value="-2.57436" />
+    <xacro:property name="limit_up_hand_rotation" value="2.57436" />
 	<!-- Links -->
     <link name="ground_link"/>
