Commit message: delete box link

File: niryo_one_description/urdf/v1/niryo_one.urdf.xacro (robot description, xacro)
@@ -16,5 +16,5 @@
 -->
 <robot xmlns:xacro="http://www.ros.org/wiki/xacro" name="niryo_one">
-	<!-- Properties -->
+     <!-- Properties -->
     <xacro:property name="distance_origin_shoulder_z" value="0.103" />
     <xacro:property name="distance_shoulder_arm_z" value="0.08" />
@@ -28,7 +28,7 @@
     <!-- not yet implemented, for now -->
     <xacro:property name="distance_hand_gripper" value="0.00" />
-	<xacro:property name="thickness_arm_axis" value="0.052" />
-	<xacro:property name="thickness_forearm_axis" value="0.048" />
-	<xacro:property name="PI" value="3.14159265359" />
+    <xacro:property name="thickness_arm_axis" value="0.052" />
+    <xacro:property name="thickness_forearm_axis" value="0.048" />
+    <xacro:property name="PI" value="3.14159265359" />
     <xacro:property name="limit_low_shoulder_rotation" value="-3.05433" />
     <xacro:property name="limit_up_shoulder_rotation" value="3.05433" />
@@ -44,244 +44,270 @@
     <xacro:property name="limit_up_hand_rotation" value="2.57" />
     <xacro:include filename="$(find niryo_one_description)/urdf/gazebo/niryo_one.gazebo.xacro" />
-	<xacro:include filename="$(find niryo_one_description)/urdf/gazebo/utils.xacro" />
-	<xacro:include filename="$(find niryo_one_description)/urdf/gazebo/niryo_one.transmission.xacro" />
-	<!-- Links -->
-	<link name="ground_link"/>
+    <xacro:include filename="$(find niryo_one_description)/urdf/gazebo/utils.xacro" />
+    <xacro:include filename="$(find niryo_one_description)/urdf/gazebo/niryo_one.transmission.xacro" />
+    <!-- Links -->
+    <link name="ground_link"/>
+    <!-- <link name="box_link">
+        <visual>
+            <origin xyz="0 0 0" rpy="0 0 0"/>
+            <geometry>
+            <box size="0.25 0.25 0.45"/>
+            </geometry>
+            <material name="Black">
+            <color rgba="0 0.0 0.0 1.0"/>
+            </material>
+        </visual>
+        <collision>
+            <origin xyz="0 0 0" rpy="0 0 0"/>
+            <geometry>
+                <box size="0.25 0.25 0.45"/>
+            </geometry>
+        </collision>
+        <inertial>
+            <mass value="1"/>
+            <inertia ixx="1.0" ixy="0.0" ixz="0.0" iyy="1.0" iyz="0.0" izz="1.0"/>
+        </inertial>
+    </link>      -->
     <link name="base_link">
-		<visual>
-			<origin xyz="0 0 0" rpy="0 0 0" />
-			<geometry>
+        <visual>
+            <origin xyz="0 0 0" rpy="0 0 0" />
+            <geometry>
                 <mesh filename="package://niryo_one_description/meshes/collada/base_link.dae" />
-			</geometry>
-			<material name="">
-				<color rgba="0.2 0.6 1 1" />
-			</material>
+            </geometry>
+            <material name="">
+               <color rgba="0.2 0.6 1 1" />
+            </material>
         </visual>
         <collision>
-			<origin xyz="0 0 0" rpy="0 0 0" />
+        <origin xyz="0 0 0" rpy="0 0 0" />
             <geometry>
                 <mesh filename="package://niryo_one_description/meshes/stl/base_link.stl" />
             </geometry>
         </collision>
-		<inertial>
-      		<origin xyz="0 0 0" rpy="0 0 0"/>
-      		<mass value="1.3"/>
-			<!--to change-->
-      		<inertia
-        		ixx="0.0" ixy="0.0" ixz="0.0"
-        		iyy="0.0" iyz="0.0"
-        		izz="0.0"/>
-    	</inertial>
-	</link>
+        <inertial>
+            <origin xyz="0 0 0" rpy="0 0 0"/>
+            <mass value="1.3"/>
+               <!--to change-->
+            <inertia
+                ixx="0.0" ixy="0.0" ixz="0.0"
+                iyy="0.0" iyz="0.0"
+                izz="0.0"/>
+            </inertial>
+    </link>
     <link name="shoulder_link">
-		<visual>
-			<origin xyz="0 0 0" rpy="0 0 0" />
-			<geometry>
+        <visual>
+            <origin xyz="0 0 0" rpy="0 0 0" />
+            <geometry>
                 <mesh filename="package://niryo_one_description/meshes/collada/shoulder_link.dae" />
-			</geometry>
-			<material name="">
-				<color rgba="0.8 0.8 0.8 1" />
-			</material>
-		</visual>
-        <collision>
-			<origin xyz="0 0 0" rpy="0 0 0" />
+            </geometry>
+            <material name="">
+                <color rgba="0.8 0.8 0.8 1" />
+            </material>
+        </visual>
+        <collision>
+            <origin xyz="0 0 0" rpy="0 0 0" />
             <geometry>
                 <mesh filename="package://niryo_one_description/meshes/stl/shoulder_link.stl" />
             </geometry>
         </collision>
-		<inertial>
-      		<origin xyz="0 0 0" rpy="0 0 0"/>
-      		<mass value="0.6"/>
-      		<inertia
-        		ixx="1.0" ixy="0.0" ixz="0.0"
-        		iyy="1.0" iyz="0.0"
-        		izz="1.0"/>
-    	</inertial>
-	</link>
+        <inertial>
+            <origin xyz="0 0 0" rpy="0 0 0"/>
+            <mass value="0.6"/>
+            <inertia
+                ixx="1.0" ixy="0.0" ixz="0.0"
+                iyy="1.0" iyz="0.0"
+                izz="1.0"/>
+            </inertial>
+    </link>
     <link name="arm_link">
-		<visual>
-			<origin xyz="0 0 0" rpy="0 0 0" />
-			<geometry>
+        <visual>
+            <origin xyz="0 0 0" rpy="0 0 0" />
+            <geometry>
                 <mesh filename="package://niryo_one_description/meshes/collada/arm_link.dae" />
-			</geometry>
-			<material name="">
-				<color rgba="0.2 0.6 1 1" />
-			</material>
-		</visual>
-        <collision>
-			<origin xyz="0 0 0" rpy="0 0 0" />
+            </geometry>
+            <material name="">
+                <color rgba="0.2 0.6 1 1" />
+            </material>
+          </visual>
+        <collision>
+               <origin xyz="0 0 0" rpy="0 0 0" />
             <geometry>
                 <mesh filename="package://niryo_one_description/meshes/stl/arm_link.stl" />
             </geometry>
         </collision>
-		<inertial>
-      		<origin xyz="0 0 0" rpy="0 0 0"/>
-      		<mass value="0.5"/>
-      		<inertia
-        		ixx="1.0" ixy="0.0" ixz="0.0"
-        		iyy="1.0" iyz="0.0"
-        		izz="1.0"/>
-    	</inertial>
-	</link>
+          <inertial>
+                <origin xyz="0 0 0" rpy="0 0 0"/>
+                <mass value="0.5"/>
+                <inertia
+                  ixx="1.0" ixy="0.0" ixz="0.0"
+                  iyy="1.0" iyz="0.0"
+                  izz="1.0"/>
+         </inertial>
+     </link>
     <link name="elbow_link">
-		<visual>
-			<origin xyz="0 0 0" rpy="0 0 0" />
-			<geometry>
-            	<!--box size="0.01 0.01 0.01"/-->
+          <visual>
+               <origin xyz="0 0 0" rpy="0 0 0" />
+               <geometry>
+                 <!--box size="0.01 0.01 0.01"/-->
                 <mesh filename="package://niryo_one_description/meshes/collada/elbow_link.dae" />
-			</geometry>
-			<material name="">
-				<color rgba="0.8 0.8 0.8 1" />
-			</material>
-		</visual>
-        <collision>
-			<origin xyz="0 0 0" rpy="0 0 0" />
+               </geometry>
+               <material name="">
+                    <color rgba="0.8 0.8 0.8 1" />
+               </material>
+          </visual>
+        <collision>
+               <origin xyz="0 0 0" rpy="0 0 0" />
             <geometry>
                 <mesh filename="package://niryo_one_description/meshes/stl/elbow_link.stl" />
             </geometry>
         </collision>
-		<inertial>
-      		<origin xyz="0 0 0" rpy="0 0 0"/>
-      		<mass value="0.4"/>
-      		<inertia
-        		ixx="1.0" ixy="0.0" ixz="0.0"
-        		iyy="1.0" iyz="0.0"
-        		izz="1.0"/>
-    	</inertial>
-	</link>
+          <inertial>
+                <origin xyz="0 0 0" rpy="0 0 0"/>
+                <mass value="0.4"/>
+                <inertia
+                  ixx="1.0" ixy="0.0" ixz="0.0"
+                  iyy="1.0" iyz="0.0"
+                  izz="1.0"/>
+         </inertial>
+     </link>
     <link name="forearm_link">
-		<visual>
-			<origin xyz="0 0 0" rpy="0 0 0" />
-			<geometry>
+          <visual>
+               <origin xyz="0 0 0" rpy="0 0 0" />
+               <geometry>
                 <mesh filename="package://niryo_one_description/meshes/collada/forearm_link.dae" />
-			</geometry>
-			<material name="">
-				<color rgba="0.2 0.6 1 1" />
-			</material>
-		</visual>
-        <collision>
-			<origin xyz="0 0 0" rpy="0 0 0" />
+               </geometry>
+               <material name="">
+                    <color rgba="0.2 0.6 1 1" />
+               </material>
+          </visual>
+        <collision>
+               <origin xyz="0 0 0" rpy="0 0 0" />
             <geometry>
                 <mesh filename="package://niryo_one_description/meshes/stl/forearm_link.stl" />
             </geometry>
         </collision>
-		<inertial>
-      		<origin xyz="0 0 0" rpy="0 0 0"/>
-      		<mass value="0.3"/>
-      		<inertia
-        		ixx="1.0" ixy="0.0" ixz="0.0"
-        		iyy="1.0" iyz="0.0"
-        		izz="1.0"/>
-    	</inertial>
-	</link>
+          <inertial>
+                <origin xyz="0 0 0" rpy="0 0 0"/>
+                <mass value="0.3"/>
+                <inertia
+                  ixx="1.0" ixy="0.0" ixz="0.0"
+                  iyy="1.0" iyz="0.0"
+                  izz="1.0"/>
+         </inertial>
+     </link>
     <link name="wrist_link">
-		<visual>
-			<origin xyz="0 0 0" rpy="0 0 0" />
-			<geometry>
+          <visual>
+               <origin xyz="0 0 0" rpy="0 0 0" />
+               <geometry>
                 <mesh filename="package://niryo_one_description/meshes/collada/wrist_link.dae" />
-			</geometry>
-			<material name="">
-				<color rgba="0.8 0.8 0.8 1" />
-			</material>
-		</visual>
-        <collision>
-			<origin xyz="0 0 0" rpy="0 0 0" />
+               </geometry>
+               <material name="">
+                    <color rgba="0.8 0.8 0.8 1" />
+               </material>
+          </visual>
+        <collision>
+               <origin xyz="0 0 0" rpy="0 0 0" />
             <geometry>
                 <mesh filename="package://niryo_one_description/meshes/stl/wrist_link.stl" />
             </geometry>
         </collision>
-		<inertial>
-      		<origin xyz="0 0 0" rpy="0 0 0"/>
-      		<mass value="0.2"/>
-      		<inertia
-        		ixx="1.0" ixy="0.0" ixz="0.0"
-        		iyy="1.0" iyz="0.0"
-        		izz="1.0"/>
-    	</inertial>
-	</link>
+          <inertial>
+                <origin xyz="0 0 0" rpy="0 0 0"/>
+                <mass value="0.2"/>
+                <inertia
+                  ixx="1.0" ixy="0.0" ixz="0.0"
+                  iyy="1.0" iyz="0.0"
+                  izz="1.0"/>
+         </inertial>
+     </link>
     <link name="hand_link">
-		<visual>
-			<origin xyz="0 0 0" rpy="0 0 0" />
-			<geometry>
+          <visual>
+               <origin xyz="0 0 0" rpy="0 0 0" />
+               <geometry>
                 <mesh filename="package://niryo_one_description/meshes/collada/hand_link.dae" />
-			</geometry>
-			<material name="">
-				<color rgba="0.6 0 0 1" />
-			</material>
-		</visual>
-        <collision>
-			<origin xyz="0 0 0" rpy="0 0 0" />
+               </geometry>
+               <material name="">
+                    <color rgba="0.6 0 0 1" />
+               </material>
+          </visual>
+        <collision>
+               <origin xyz="0 0 0" rpy="0 0 0" />
             <geometry>
                 <mesh filename="package://niryo_one_description/meshes/stl/hand_link.stl" />
             </geometry>
         </collision>
-		<inertial>
-      		<origin xyz="0 0 0" rpy="0 0 0"/>
-      		<mass value="0.1"/>
-      		<inertia
-        		ixx="1.0" ixy="0.0" ixz="0.0"
-        		iyy="1.0" iyz="0.0"
-        		izz="1.0"/>
-    	</inertial>
-	</link>
+          <inertial>
+                <origin xyz="0 0 0" rpy="0 0 0"/>
+                <mass value="0.1"/>
+                <inertia
+                  ixx="1.0" ixy="0.0" ixz="0.0"
+                  iyy="1.0" iyz="0.0"
+                  izz="1.0"/>
+         </inertial>
+     </link>
     <link name="gripper_link">
-	</link>
-	<!--Joints -->
-	<joint name="ground_joint" type="fixed">
+     </link>
+     <!--Joints -->
+     <!-- <joint name="ground_joint" type="fixed">
+        <parent link="ground_link" />
+        <child link="box_link" />
+        <origin xyz="0.0 0.0 0.0" rpy="0 0 0" />
+    </joint> -->
+    <joint name="ground_joint" type="fixed">
         <parent link="ground_link" />
         <child link="base_link" />
-        <origin xyz="0.0 0.0 0.0" rpy="0 0 0" />
-    </joint>
-	<joint name="joint_1" type="revolute">
+        <origin xyz="0.0 0.0 0" rpy="0 0 0" />
+    </joint>
+    <joint name="joint_1" type="revolute">
         <parent link="base_link" />
         <child link="shoulder_link" />
-		<origin xyz="0 0 ${distance_origin_shoulder_z}" rpy="0 0 0" />
-		<axis xyz="0 0 1" />
-		<limit effort="1" velocity="1.0" lower="${limit_low_shoulder_rotation}" upper="${limit_up_shoulder_rotation}" />
-	</joint>
-	<joint name="joint_2" type="revolute">
+          <origin xyz="0 0 ${distance_origin_shoulder_z}" rpy="0 0 0" />
+          <axis xyz="0 0 1" />
+          <limit effort="1" velocity="1.0" lower="${limit_low_shoulder_rotation}" upper="${limit_up_shoulder_rotation}" />
+    </joint>
+    <joint name="joint_2" type="revolute">
         <parent link="shoulder_link" />
         <child link="arm_link" />
         <origin xyz="0 0 ${distance_shoulder_arm_z}" rpy="${PI/2} ${-PI/2} 0" />
-		<limit effort="1" velocity="1.0" lower="${limit_low_arm_rotation}" upper="${limit_up_arm_rotation}" />
-		<axis xyz="0 0 1" />
-	</joint>
-	<joint name="joint_3" type="revolute">
+          <limit effort="1" velocity="1.0" lower="${limit_low_arm_rotation}" upper="${limit_up_arm_rotation}" />
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
File: niryo_one_description/urdf/v1/without_mesh_niryo_one.urdf.xacro (robot description, xacro)
@@ -16,7 +16,7 @@
 -->
 <robot xmlns:xacro="http://www.ros.org/wiki/xacro" name="niryo_one">
-	<!-- Properties -->
-	<xacro:property name="distance_origin_shoulder_z" value="0.103" />
-	<xacro:property name="distance_shoulder_arm_z" value="0.08" />
+     <!-- Properties -->
+    <xacro:property name="distance_origin_shoulder_z" value="0.103" />
+    <xacro:property name="distance_shoulder_arm_z" value="0.08" />
     <xacro:property name="distance_arm_elbow_x" value="0.21004" />
     <xacro:property name="distance_arm_elbow_y" value="0.0" />
@@ -24,13 +24,13 @@
     <xacro:property name="distance_elbow_forearm_y" value="0.032" />
     <xacro:property name="distance_forearm_wrist_z" value="0.180" />
-	<xacro:property name="distance_wrist_hand_x" value="0.018" />
+    <xacro:property name="distance_wrist_hand_x" value="0.018" />
     <xacro:property name="distance_wrist_hand_y" value="0" />
     <!-- not yet implemented, tools are handled separately -->
     <xacro:property name="distance_hand_gripper" value="0.00" />
-	<xacro:property name="thickness_arm_axis" value="0.052" />
-	<xacro:property name="thickness_forearm_axis" value="0.048" />
-	<xacro:property name="PI" value="3.14159265359" />
-	<xacro:property name="limit_low_shoulder_rotation" value="-3.05433" />
-	<xacro:property name="limit_up_shoulder_rotation" value="3.05433" />
+    <xacro:property name="thickness_arm_axis" value="0.052" />
+    <xacro:property name="thickness_forearm_axis" value="0.048" />
+    <xacro:property name="PI" value="3.14159265359" />
+    <xacro:property name="limit_low_shoulder_rotation" value="-3.05433" />
+    <xacro:property name="limit_up_shoulder_rotation" value="3.05433" />
     <xacro:property name="limit_low_arm_rotation" value="${-PI/2}" />
     <xacro:property name="limit_up_arm_rotation" value="0.628319" />
@@ -43,23 +43,23 @@
     <xacro:property name="limit_low_hand_rotation" value="-2.57" />
     <xacro:property name="limit_up_hand_rotation" value="2.57" />
-	<!-- Links -->
+     <!-- Links -->
     <link name="ground_link"/>
     <link name="base_link">
-	</link>
+    </link>
     <link name="shoulder_link">
-	</link>
+    </link>
     <link name="arm_link">
-	</link>
+    </link>
     <link name="elbow_link">
-	</link>
+    </link>
     <link name="forearm_link">
-	</link>
+    </link>
     <link name="wrist_link">
-	</link>
+    </link>
     <link name="hand_link">
-	</link>
+    </link>
     <link name="gripper_link">
-	</link>
-	<!--Joints -->
+    </link>
+     <!--Joints -->
     <joint name="ground_joint" type="fixed">
         <parent link="ground_link" />
@@ -67,50 +67,50 @@
         <origin xyz="0 0 0" rpy="0 0 0" />
     </joint>
-	<joint name="joint_1" type="revolute">
+    <joint name="joint_1" type="revolute">
         <parent link="base_link" />
         <child link="shoulder_link" />
-		<origin xyz="0 0 ${distance_origin_shoulder_z}" rpy="0 0 0" />
-		<axis xyz="0 0 1" />
-		<limit effort="1" velocity="1.0" lower="${limit_low_shoulder_rotation}" upper="${limit_up_shoulder_rotation}" />
-	</joint>
-	<joint name="joint_2" type="revolute">
+          <origin xyz="0 0 ${distance_origin_shoulder_z}" rpy="0 0 0" />
+          <axis xyz="0 0 1" />
+          <limit effort="1" velocity="1.0" lower="${limit_low_shoulder_rotation}" upper="${limit_up_shoulder_rotation}" />
+    </joint>
+    <joint name="joint_2" type="revolute">
         <parent link="shoulder_link" />
         <child link="arm_link" />
         <origin xyz="0 0 ${distance_shoulder_arm_z}" rpy="${PI/2} ${-PI/2} 0" />
-		<limit effort="1" velocity="1.0" lower="${limit_low_arm_rotation}" upper="${limit_up_arm_rotation}" />
-		<axis xyz="0 0 1" />
-	</joint>
-	<joint name="joint_3" type="revolute">
+          <limit effort="1" velocity="1.0" lower="${limit_low_arm_rotation}" upper="${limit_up_arm_rotation}" />
+          <axis xyz="0 0 1" />
+    </joint>
+    <joint name="joint_3" type="revolute">
         <parent link="arm_link" />
         <child link="elbow_link" />
         <origin xyz="${distance_arm_elbow_x} ${distance_arm_elbow_y} 0" rpy="0 0 ${-PI/2}" />
-		<limit effort="1" velocity="1.0" lower="${limit_low_elbow_rotation}" upper="${limit_up_elbow_rotation}" />
-		<axis xyz="0 0 1" />
-	</joint>
-	<joint name="joint_4" type="revolute">
+          <limit effort="1" velocity="1.0" lower="${limit_low_elbow_rotation}" upper="${limit_up_elbow_rotation}" />
+          <axis xyz="0 0 1" />
+    </joint>
+    <joint name="joint_4" type="revolute">
         <parent link="elbow_link" />
         <child link="forearm_link" />
         <origin xyz="${distance_elbow_forearm_x} ${distance_elbow_forearm_y} 0" rpy="0 ${PI/2} 0" />
-		<limit effort="1" velocity="1.0" lower="${limit_low_forearm_rotation}" upper="${limit_up_forearm_rotation}" />
-		<axis xyz="0 0 1" />
-	</joint>
-	<joint name="joint_5" type="revolute">
+          <limit effort="1" velocity="1.0" lower="${limit_low_forearm_rotation}" upper="${limit_up_forearm_rotation}" />
+          <axis xyz="0 0 1" />
+    </joint>
+    <joint name="joint_5" type="revolute">
         <parent link="forearm_link" />
         <child link="wrist_link" />
-		<origin xyz="0 0 ${distance_forearm_wrist_z}" rpy="0 ${-PI/2} 0" />
-		<limit effort="1" velocity="1.0" lower="${limit_low_wrist_rotation}" upper="${limit_up_wrist_rotation}" />
-		<axis xyz="0 0 1" />
-	</joint>
-	<joint name="joint_6" type="revolute">
+          <origin xyz="0 0 ${distance_forearm_wrist_z}" rpy="0 ${-PI/2} 0" />
+          <limit effort="1" velocity="1.0" lower="${limit_low_wrist_rotation}" upper="${limit_up_wrist_rotation}" />
+          <axis xyz="0 0 1" />
+    </joint>
+    <joint name="joint_6" type="revolute">
         <parent link="wrist_link" />
         <child link="hand_link" />
         <origin xyz="${distance_wrist_hand_x} ${distance_wrist_hand_y} 0" rpy="0 ${PI/2} 0" />
-		<limit effort="1" velocity="1.0" lower="${limit_low_hand_rotation}" upper="${limit_up_hand_rotation}" />
-		<axis xyz="0 0 1" />
-	</joint>
-	<joint name="hand_gripper_joint" type="fixed">
+          <limit effort="1" velocity="1.0" lower="${limit_low_hand_rotation}" upper="${limit_up_hand_rotation}" />
+          <axis xyz="0 0 1" />
+    </joint>
+    <joint name="hand_gripper_joint" type="fixed">
         <parent link="hand_link" />
         <child link="gripper_link" />
         <origin xyz="0 0 ${distance_hand_gripper}" rpy="${-PI/2} ${-PI/2} 0" />
-	</joint>
+    </joint>
 </robot>
