Commit message: fix merge conflicts

File: niryo_one_description/urdf/v1/niryo_one.urdf.xacro (robot description, xacro)
@@ -26,14 +26,6 @@
     <xacro:property name="distance_wrist_hand_x" value="0.018" />
     <xacro:property name="distance_wrist_hand_y" value="0" />
-<<<<<<< HEAD
-    <!-- not yet implemented, for now -->
-    <xacro:property name="distance_hand_gripper" value="0.00" />
-    <xacro:property name="thickness_arm_axis" value="0.052" />
-    <xacro:property name="thickness_forearm_axis" value="0.048" />
-    <xacro:property name="PI" value="3.14159265359" />
-=======
     <xacro:property name="distance_hand_tool" value="0.00" />
 	<xacro:property name="PI" value="3.14159265359" />
->>>>>>> f9562b7a28424a0d9a25d0dd6343b672fabdfdae
     <xacro:property name="limit_low_shoulder_rotation" value="-3.05433" />
     <xacro:property name="limit_up_shoulder_rotation" value="3.05433" />
@@ -75,14 +67,4 @@
     </link>      -->
     <link name="base_link">
-<<<<<<< HEAD
-        <visual>
-            <origin xyz="0 0 0" rpy="0 0 0" />
-            <geometry>
-                <mesh filename="package://niryo_one_description/meshes/collada/base_link.dae" />
-            </geometry>
-            <material name="">
-               <color rgba="0.2 0.6 1 1" />
-            </material>
-=======
 		<visual>
 			<origin xyz="0 0 0" rpy="0 0 0" />
@@ -93,5 +75,4 @@
 				<color rgba="0.2 0.6 1 1" />
 			</material>
->>>>>>> f9562b7a28424a0d9a25d0dd6343b672fabdfdae
         </visual>
         <collision>
@@ -112,28 +93,16 @@
     </link>
     <link name="shoulder_link">
-<<<<<<< HEAD
-        <visual>
+		<visual>
+			<origin xyz="0 0 0" rpy="0 0 0" />
+			<geometry>
+                <mesh filename="package://niryo_one_description/meshes/v1/collada/shoulder_link.dae" />
+			</geometry>
+			<material name="">
+				<color rgba="0.8 0.8 0.8 1" />
+			</material>
+		</visual>
+        <collision>
             <origin xyz="0 0 0" rpy="0 0 0" />
             <geometry>
-                <mesh filename="package://niryo_one_description/meshes/collada/shoulder_link.dae" />
-            </geometry>
-            <material name="">
-                <color rgba="0.8 0.8 0.8 1" />
-            </material>
-        </visual>
-=======
-		<visual>
-			<origin xyz="0 0 0" rpy="0 0 0" />
-			<geometry>
-                <mesh filename="package://niryo_one_description/meshes/v1/collada/shoulder_link.dae" />
-			</geometry>
-			<material name="">
-				<color rgba="0.8 0.8 0.8 1" />
-			</material>
-		</visual>
->>>>>>> f9562b7a28424a0d9a25d0dd6343b672fabdfdae
-        <collision>
-            <origin xyz="0 0 0" rpy="0 0 0" />
-            <geometry>
                 <mesh filename="package://niryo_one_description/meshes/v1/stl/shoulder_link.stl" />
             </geometry>
@@ -146,18 +115,7 @@
                 iyy="1.0" iyz="0.0"
                 izz="1.0"/>
-            </inertial>
+        </inertial>
     </link>
     <link name="arm_link">
-<<<<<<< HEAD
-        <visual>
-            <origin xyz="0 0 0" rpy="0 0 0" />
-            <geometry>
-                <mesh filename="package://niryo_one_description/meshes/collada/arm_link.dae" />
-            </geometry>
-            <material name="">
-                <color rgba="0.2 0.6 1 1" />
-            </material>
-          </visual>
-=======
 		<visual>
 			<origin xyz="0 0 0" rpy="0 0 0" />
@@ -169,5 +127,4 @@
 			</material>
 		</visual>
->>>>>>> f9562b7a28424a0d9a25d0dd6343b672fabdfdae
         <collision>
                <origin xyz="0 0 0" rpy="0 0 0" />
@@ -176,26 +133,14 @@
             </geometry>
         </collision>
-          <inertial>
-                <origin xyz="0 0 0" rpy="0 0 0"/>
-                <mass value="0.5"/>
-                <inertia
-                  ixx="1.0" ixy="0.0" ixz="0.0"
-                  iyy="1.0" iyz="0.0"
-                  izz="1.0"/>
-         </inertial>
-     </link>
+        <inertial>
+            <origin xyz="0 0 0" rpy="0 0 0"/>
+            <mass value="0.5"/>
+            <inertia
+                ixx="1.0" ixy="0.0" ixz="0.0"
+                iyy="1.0" iyz="0.0"
+                izz="1.0"/>
+        </inertial>
+    </link>
     <link name="elbow_link">
-<<<<<<< HEAD
-          <visual>
-               <origin xyz="0 0 0" rpy="0 0 0" />
-               <geometry>
-                 <!--box size="0.01 0.01 0.01"/-->
-                <mesh filename="package://niryo_one_description/meshes/collada/elbow_link.dae" />
-               </geometry>
-               <material name="">
-                    <color rgba="0.8 0.8 0.8 1" />
-               </material>
-          </visual>
-=======
 		<visual>
 			<origin xyz="0 0 0" rpy="0 0 0" />
@@ -208,5 +153,4 @@
 			</material>
 		</visual>
->>>>>>> f9562b7a28424a0d9a25d0dd6343b672fabdfdae
         <collision>
                <origin xyz="0 0 0" rpy="0 0 0" />
@@ -215,25 +159,14 @@
             </geometry>
         </collision>
-          <inertial>
-                <origin xyz="0 0 0" rpy="0 0 0"/>
-                <mass value="0.4"/>
-                <inertia
-                  ixx="1.0" ixy="0.0" ixz="0.0"
-                  iyy="1.0" iyz="0.0"
-                  izz="1.0"/>
-         </inertial>
-     </link>
+        <inertial>
+            <origin xyz="0 0 0" rpy="0 0 0"/>
+            <mass value="0.4"/>
+            <inertia
+                ixx="1.0" ixy="0.0" ixz="0.0"
+                iyy="1.0" iyz="0.0"
+                izz="1.0"/>
+        </inertial>
+    </link>
     <link name="forearm_link">
-<<<<<<< HEAD
-          <visual>
-               <origin xyz="0 0 0" rpy="0 0 0" />
-               <geometry>
-                <mesh filename="package://niryo_one_description/meshes/collada/forearm_link.dae" />
-               </geometry>
-               <material name="">
-                    <color rgba="0.2 0.6 1 1" />
-               </material>
-          </visual>
-=======
 		<visual>
 			<origin xyz="0 0 0" rpy="0 0 0" />
@@ -245,5 +178,4 @@
 			</material>
 		</visual>
->>>>>>> f9562b7a28424a0d9a25d0dd6343b672fabdfdae
         <collision>
                <origin xyz="0 0 0" rpy="0 0 0" />
@@ -252,25 +184,14 @@
             </geometry>
         </collision>
-          <inertial>
-                <origin xyz="0 0 0" rpy="0 0 0"/>
-                <mass value="0.3"/>
-                <inertia
-                  ixx="1.0" ixy="0.0" ixz="0.0"
-                  iyy="1.0" iyz="0.0"
-                  izz="1.0"/>
-         </inertial>
-     </link>
+        <inertial>
+            <origin xyz="0 0 0" rpy="0 0 0"/>
+            <mass value="0.3"/>
+            <inertia
+                ixx="1.0" ixy="0.0" ixz="0.0"
+                iyy="1.0" iyz="0.0"
+                izz="1.0"/>
+        </inertial>
+    </link>
     <link name="wrist_link">
-<<<<<<< HEAD
-          <visual>
-               <origin xyz="0 0 0" rpy="0 0 0" />
-               <geometry>
-                <mesh filename="package://niryo_one_description/meshes/collada/wrist_link.dae" />
-               </geometry>
-               <material name="">
-                    <color rgba="0.8 0.8 0.8 1" />
-               </material>
-          </visual>
-=======
 		<visual>
 			<origin xyz="0 0 0" rpy="0 0 0" />
@@ -282,5 +203,4 @@
 			</material>
 		</visual>
->>>>>>> f9562b7a28424a0d9a25d0dd6343b672fabdfdae
         <collision>
                <origin xyz="0 0 0" rpy="0 0 0" />
@@ -289,25 +209,14 @@
             </geometry>
         </collision>
-          <inertial>
-                <origin xyz="0 0 0" rpy="0 0 0"/>
-                <mass value="0.2"/>
-                <inertia
-                  ixx="1.0" ixy="0.0" ixz="0.0"
-                  iyy="1.0" iyz="0.0"
-                  izz="1.0"/>
-         </inertial>
-     </link>
+        <inertial>
+            <origin xyz="0 0 0" rpy="0 0 0"/>
+            <mass value="0.2"/>
+            <inertia
+                ixx="1.0" ixy="0.0" ixz="0.0"
+                iyy="1.0" iyz="0.0"
+                izz="1.0"/>
+        </inertial>
+    </link>
     <link name="hand_link">
-<<<<<<< HEAD
-          <visual>
-               <origin xyz="0 0 0" rpy="0 0 0" />
-               <geometry>
-                <mesh filename="package://niryo_one_description/meshes/collada/hand_link.dae" />
-               </geometry>
-               <material name="">
-                    <color rgba="0.6 0 0 1" />
-               </material>
-          </visual>
-=======
 		<visual>
 			<origin xyz="0 0 0" rpy="0 0 0" />
@@ -319,5 +228,4 @@
 			</material>
 		</visual>
->>>>>>> f9562b7a28424a0d9a25d0dd6343b672fabdfdae
         <collision>
                <origin xyz="0 0 0" rpy="0 0 0" />
@@ -326,5 +234,4 @@
             </geometry>
         </collision>
-<<<<<<< HEAD
           <inertial>
                 <origin xyz="0 0 0" rpy="0 0 0"/>
@@ -336,11 +243,6 @@
          </inertial>
      </link>
-    <link name="gripper_link">
-     </link>
-=======
-	</link>
     <link name="tool_link">
 	</link>
->>>>>>> f9562b7a28424a0d9a25d0dd6343b672fabdfdae
      <!--Joints -->
      <!-- <joint name="ground_joint" type="fixed">
@@ -396,10 +298,9 @@
           <axis xyz="0 0 1" />
 	</joint>
-<<<<<<< HEAD
-    <joint name="hand_gripper_joint" type="fixed">
+    <joint name="hand_tool_joint" type="fixed">
         <parent link="hand_link" />
-        <child link="gripper_link" />
-        <origin xyz="0 0 ${distance_hand_gripper}" rpy="${-PI/2} ${-PI/2} 0" />
-    </joint>
+        <child link="tool_link" />
+        <origin xyz="0 0 ${distance_hand_tool}" rpy="${-PI/2} ${-PI/2} 0" />
+	</joint>
      <!--plugin-->
     <gazebo>
@@ -407,10 +308,3 @@
             </plugin>
     </gazebo>
-=======
-	<joint name="hand_tool_joint" type="fixed">
-        <parent link="hand_link" />
-        <child link="tool_link" />
-        <origin xyz="0 0 ${distance_hand_tool}" rpy="${-PI/2} ${-PI/2} 0" />
-	</joint>
->>>>>>> f9562b7a28424a0d9a25d0dd6343b672fabdfdae
 </robot>
