Commit message: Gazebo simulator (#22)
* create gazebo aspects of niryo and add it to urdf file

* create gaezbo package and world

* change color tag

* add transmission tag for robot control

* launch file for gazebo and controller nodes

* add robot_commander node and others node to gazebo launch file

* organize xacro gazebo files

* include niryo_one_base in niryo_one_gazebo.launch

* clean files

* add hardware version v2 to gazebo simulation

* change controllers constraints

*  add gazeon models

*  add gazebo xacro model description

* delete box link

* no include gazebo convoyer model

*  add camera to gazebo world and fix file position manager

*  fix merge conflicts

* comment camera section

* comment gazebo colors to use stl colors

* keep defanut version v2 when launching gazebo simulation

*  restore niryo_one V1 colors

* update gazebo simulation with ros melodic

*  add README section about gazebo simulation

* Update README

* add tf2 node

* change iryo_one_gazebo version to V2.1.0

* refactor some files

*  delete a log file

* add licence text to some files

File: niryo_one_description/urdf/v1/niryo_one.urdf.xacro (robot description, xacro)
@@ -16,5 +16,5 @@
 -->
 <robot xmlns:xacro="http://www.ros.org/wiki/xacro" name="niryo_one">
-	<!-- Properties -->
+     <!-- Properties -->
     <xacro:property name="distance_origin_shoulder_z" value="0.103" />
     <xacro:property name="distance_shoulder_arm_z" value="0.08" />
@@ -40,6 +40,30 @@
     <xacro:property name="limit_low_hand_rotation" value="-2.57" />
     <xacro:property name="limit_up_hand_rotation" value="2.57" />
-	<!-- Links -->
+    <xacro:include filename="$(find niryo_one_description)/urdf/gazebo/niryo_one_v1.gazebo.xacro" />
+    <xacro:include filename="$(find niryo_one_description)/urdf/gazebo/utils.xacro" />
+    <xacro:include filename="$(find niryo_one_description)/urdf/gazebo/niryo_one.transmission.xacro" />
+    <!-- Links -->
     <link name="ground_link"/>
+    <!-- <link name="box_link">
+        <visual>
+            <origin xyz="0 0 0" rpy="0 0 0"/>
+            <geometry>
+            <box size="0.25 0.25 0.45"/>
+            </geometry>
+            <material name="Black">
+            <color rgba="0 0.0 0.0 1.0"/>
+            </material>
+        </visual>
+        <collision>
+            <origin xyz="0 0 0" rpy="0 0 0"/>
+            <geometry>
+                <box size="0.25 0.25 0.45"/>
+            </geometry>
+        </collision>
+        <inertial>
+            <mass value="1"/>
+            <inertia ixx="1.0" ixy="0.0" ixz="0.0" iyy="1.0" iyz="0.0" izz="1.0"/>
+        </inertial>
+    </link>      -->
     <link name="base_link">
 		<visual>
@@ -53,10 +77,19 @@
         </visual>
         <collision>
-			<origin xyz="0 0 0" rpy="0 0 0" />
+        <origin xyz="0 0 0" rpy="0 0 0" />
             <geometry>
                 <mesh filename="package://niryo_one_description/meshes/v1/stl/base_link.stl" />
             </geometry>
         </collision>
-	</link>
+        <inertial>
+            <origin xyz="0 0 0" rpy="0 0 0"/>
+            <mass value="1.3"/>
+               <!--to change-->
+            <inertia
+                ixx="0.0" ixy="0.0" ixz="0.0"
+                iyy="0.0" iyz="0.0"
+                izz="0.0"/>
+            </inertial>
+    </link>
     <link name="shoulder_link">
 		<visual>
@@ -70,10 +103,18 @@
 		</visual>
         <collision>
-			<origin xyz="0 0 0" rpy="0 0 0" />
+            <origin xyz="0 0 0" rpy="0 0 0" />
             <geometry>
                 <mesh filename="package://niryo_one_description/meshes/v1/stl/shoulder_link.stl" />
             </geometry>
         </collision>
-	</link>
+        <inertial>
+            <origin xyz="0 0 0" rpy="0 0 0"/>
+            <mass value="0.6"/>
+            <inertia
+                ixx="1.0" ixy="0.0" ixz="0.0"
+                iyy="1.0" iyz="0.0"
+                izz="1.0"/>
+        </inertial>
+    </link>
     <link name="arm_link">
 		<visual>
@@ -87,10 +128,18 @@
 		</visual>
         <collision>
-			<origin xyz="0 0 0" rpy="0 0 0" />
+               <origin xyz="0 0 0" rpy="0 0 0" />
             <geometry>
                 <mesh filename="package://niryo_one_description/meshes/v1/stl/arm_link.stl" />
             </geometry>
         </collision>
-	</link>
+        <inertial>
+            <origin xyz="0 0 0" rpy="0 0 0"/>
+            <mass value="0.5"/>
+            <inertia
+                ixx="1.0" ixy="0.0" ixz="0.0"
+                iyy="1.0" iyz="0.0"
+                izz="1.0"/>
+        </inertial>
+    </link>
     <link name="elbow_link">
 		<visual>
@@ -105,10 +154,18 @@
 		</visual>
         <collision>
-			<origin xyz="0 0 0" rpy="0 0 0" />
+               <origin xyz="0 0 0" rpy="0 0 0" />
             <geometry>
                 <mesh filename="package://niryo_one_description/meshes/v1/stl/elbow_link.stl" />
             </geometry>
         </collision>
-	</link>
+        <inertial>
+            <origin xyz="0 0 0" rpy="0 0 0"/>
+            <mass value="0.4"/>
+            <inertia
+                ixx="1.0" ixy="0.0" ixz="0.0"
+                iyy="1.0" iyz="0.0"
+                izz="1.0"/>
+        </inertial>
+    </link>
     <link name="forearm_link">
 		<visual>
@@ -122,10 +179,18 @@
 		</visual>
         <collision>
-			<origin xyz="0 0 0" rpy="0 0 0" />
+               <origin xyz="0 0 0" rpy="0 0 0" />
             <geometry>
                 <mesh filename="package://niryo_one_description/meshes/v1/stl/forearm_link.stl" />
             </geometry>
         </collision>
-	</link>
+        <inertial>
+            <origin xyz="0 0 0" rpy="0 0 0"/>
+            <mass value="0.3"/>
+            <inertia
+                ixx="1.0" ixy="0.0" ixz="0.0"
+                iyy="1.0" iyz="0.0"
+                izz="1.0"/>
+        </inertial>
+    </link>
     <link name="wrist_link">
 		<visual>
@@ -139,10 +204,18 @@
 		</visual>
         <collision>
-			<origin xyz="0 0 0" rpy="0 0 0" />
+               <origin xyz="0 0 0" rpy="0 0 0" />
             <geometry>
                 <mesh filename="package://niryo_one_description/meshes/v1/stl/wrist_link.stl" />
             </geometry>
         </collision>
-	</link>
+        <inertial>
+            <origin xyz="0 0 0" rpy="0 0 0"/>
+            <mass value="0.2"/>
+            <inertia
+                ixx="1.0" ixy="0.0" ixz="0.0"
+                iyy="1.0" iyz="0.0"
+                izz="1.0"/>
+        </inertial>
+    </link>
     <link name="hand_link">
 		<visual>
@@ -156,64 +229,82 @@
 		</visual>
         <collision>
-			<origin xyz="0 0 0" rpy="0 0 0" />
+               <origin xyz="0 0 0" rpy="0 0 0" />
             <geometry>
                 <mesh filename="package://niryo_one_description/meshes/v1/stl/hand_link.stl" />
             </geometry>
         </collision>
-	</link>
+          <inertial>
+                <origin xyz="0 0 0" rpy="0 0 0"/>
+                <mass value="0.1"/>
+                <inertia
+                  ixx="1.0" ixy="0.0" ixz="0.0"
+                  iyy="1.0" iyz="0.0"
+                  izz="1.0"/>
+         </inertial>
+     </link>
     <link name="tool_link">
 	</link>
-	<!--Joints -->
+     <!--Joints -->
+     <!-- <joint name="ground_joint" type="fixed">
+        <parent link="ground_link" />
+        <child link="box_link" />
+        <origin xyz="0.0 0.0 0.0" rpy="0 0 0" />
+    </joint> -->
     <joint name="ground_joint" type="fixed">
         <parent link="ground_link" />
         <child link="base_link" />
-        <origin xyz="0 0 0" rpy="0 0 0" />
-    </joint>
-	<joint name="joint_1" type="revolute">
+        <origin xyz="0.0 0.0 0" rpy="0 0 0" />
+    </joint>
+    <joint name="joint_1" type="revolute">
         <parent link="base_link" />
         <child link="shoulder_link" />
-		<origin xyz="0 0 ${distance_origin_shoulder_z}" rpy="0 0 0" />
-		<axis xyz="0 0 1" />
-		<limit effort="1" velocity="1.0" lower="${limit_low_shoulder_rotation}" upper="${limit_up_shoulder_rotation}" />
-	</joint>
-	<joint name="joint_2" type="revolute">
+          <origin xyz="0 0 ${distance_origin_shoulder_z}" rpy="0 0 0" />
+          <axis xyz="0 0 1" />
+          <limit effort="1" velocity="1.0" lower="${limit_low_shoulder_rotation}" upper="${limit_up_shoulder_rotation}" />
+    </joint>
+    <joint name="joint_2" type="revolute">
         <parent link="shoulder_link" />
         <child link="arm_link" />
         <origin xyz="0 0 ${distance_shoulder_arm_z}" rpy="${PI/2} ${-PI/2} 0" />
-		<limit effort="1" velocity="1.0" lower="${limit_low_arm_rotation}" upper="${limit_up_arm_rotation}" />
-		<axis xyz="0 0 1" />
-	</joint>
-	<joint name="joint_3" type="revolute">
+          <limit effort="1" velocity="1.0" lower="${limit_low_arm_rotation}" upper="${limit_up_arm_rotation}" />
+          <axis xyz="0 0 1" />
+    </joint>
+    <joint name="joint_3" type="revolute">
         <parent link="arm_link" />
         <child link="elbow_link" />
         <origin xyz="${distance_arm_elbow_x} ${distance_arm_elbow_y} 0" rpy="0 0 ${-PI/2}" />
-		<limit effort="1" velocity="1.0" lower="${limit_low_elbow_rotation}" upper="${limit_up_elbow_rotation}" />
-		<axis xyz="0 0 1" />
-	</joint>
-	<joint name="joint_4" type="revolute">
+          <limit effort="1" velocity="1.0" lower="${limit_low_elbow_rotation}" upper="${limit_up_elbow_rotation}" />
+          <axis xyz="0 0 1" />
+    </joint>
+    <joint name="joint_4" type="revolute">
         <parent link="elbow_link" />
         <child link="forearm_link" />
         <origin xyz="${distance_elbow_forearm_x} ${distance_elbow_forearm_y} 0" rpy="0 ${PI/2} 0" />
-		<limit effort="1" velocity="1.0" lower="${limit_low_forearm_rotation}" upper="${limit_up_forearm_rotation}" />
-		<axis xyz="0 0 1" />
-	</joint>
-	<joint name="joint_5" type="revolute">
+          <limit effort="1" velocity="1.0" lower="${limit_low_forearm_rotation}" upper="${limit_up_forearm_rotation}" />
+          <axis xyz="0 0 1" />
+    </joint>
+    <joint name="joint_5" type="revolute">
         <parent link="forearm_link" />
         <child link="wrist_link" />
-		<origin xyz="0 0 ${distance_forearm_wrist_z}" rpy="0 ${-PI/2} 0" />
-		<limit effort="1" velocity="1.0" lower="${limit_low_wrist_rotation}" upper="${limit_up_wrist_rotation}" />
-		<axis xyz="0 0 1" />
-	</joint>
-	<joint name="joint_6" type="revolute">
+          <origin xyz="0 0 ${distance_forearm_wrist_z}" rpy="0 ${-PI/2} 0" />
+          <limit effort="1" velocity="1.0" lower="${limit_low_wrist_rotation}" upper="${limit_up_wrist_rotation}" />
+          <axis xyz="0 0 1" />
+    </joint>
+    <joint name="joint_6" type="revolute">
         <parent link="wrist_link" />
         <child link="hand_link" />
         <origin xyz="${distance_wrist_hand_x} ${distance_wrist_hand_y} 0" rpy="0 ${PI/2} 0" />
-		<limit effort="1" velocity="1.0" lower="${limit_low_hand_rotation}" upper="${limit_up_hand_rotation}" />
-		<axis xyz="0 0 1" />
+          <limit effort="1" velocity="1.0" lower="${limit_low_hand_rotation}" upper="${limit_up_hand_rotation}" />
+          <axis xyz="0 0 1" />
 	</joint>
-	<joint name="hand_tool_joint" type="fixed">
+    <joint name="hand_tool_joint" type="fixed">
         <parent link="hand_link" />
         <child link="tool_link" />
         <origin xyz="0 0 ${distance_hand_tool}" rpy="${-PI/2} ${-PI/2} 0" />
 	</joint>
+     <!--plugin-->
+    <gazebo>
+            <plugin name="gazebo_ros_control" filename="libgazebo_ros_control.so">
+            </plugin>
+    </gazebo>
 </robot>

File: niryo_one_description/urdf/v1/without_mesh_niryo_one.urdf.xacro (robot description, xacro)
@@ -16,7 +16,7 @@
 -->
 <robot xmlns:xacro="http://www.ros.org/wiki/xacro" name="niryo_one">
-	<!-- Properties -->
-	<xacro:property name="distance_origin_shoulder_z" value="0.103" />
-	<xacro:property name="distance_shoulder_arm_z" value="0.08" />
+     <!-- Properties -->
+    <xacro:property name="distance_origin_shoulder_z" value="0.103" />
+    <xacro:property name="distance_shoulder_arm_z" value="0.08" />
     <xacro:property name="distance_arm_elbow_x" value="0.21004" />
     <xacro:property name="distance_arm_elbow_y" value="0.0" />
@@ -24,5 +24,5 @@
     <xacro:property name="distance_elbow_forearm_y" value="0.032" />
     <xacro:property name="distance_forearm_wrist_z" value="0.180" />
-	<xacro:property name="distance_wrist_hand_x" value="0.018" />
+    <xacro:property name="distance_wrist_hand_x" value="0.018" />
     <xacro:property name="distance_wrist_hand_y" value="0" />
     <xacro:property name="distance_hand_tool" value="0.00" />
@@ -40,23 +40,23 @@
     <xacro:property name="limit_low_hand_rotation" value="-2.57" />
     <xacro:property name="limit_up_hand_rotation" value="2.57" />
-	<!-- Links -->
+     <!-- Links -->
     <link name="ground_link"/>
     <link name="base_link">
-	</link>
+    </link>
     <link name="shoulder_link">
-	</link>
+    </link>
     <link name="arm_link">
-	</link>
+    </link>
     <link name="elbow_link">
-	</link>
+    </link>
     <link name="forearm_link">
-	</link>
+    </link>
     <link name="wrist_link">
-	</link>
+    </link>
     <link name="hand_link">
 	</link>
     <link name="tool_link">
 	</link>
-	<!--Joints -->
+     <!--Joints -->
     <joint name="ground_joint" type="fixed">
         <parent link="ground_link" />
@@ -64,46 +64,46 @@
         <origin xyz="0 0 0" rpy="0 0 0" />
     </joint>
-	<joint name="joint_1" type="revolute">
+    <joint name="joint_1" type="revolute">
         <parent link="base_link" />
         <child link="shoulder_link" />
-		<origin xyz="0 0 ${distance_origin_shoulder_z}" rpy="0 0 0" />
-		<axis xyz="0 0 1" />
-		<limit effort="1" velocity="1.0" lower="${limit_low_shoulder_rotation}" upper="${limit_up_shoulder_rotation}" />
-	</joint>
-	<joint name="joint_2" type="revolute">
+          <origin xyz="0 0 ${distance_origin_shoulder_z}" rpy="0 0 0" />
+          <axis xyz="0 0 1" />
+          <limit effort="1" velocity="1.0" lower="${limit_low_shoulder_rotation}" upper="${limit_up_shoulder_rotation}" />
+    </joint>
+    <joint name="joint_2" type="revolute">
         <parent link="shoulder_link" />
         <child link="arm_link" />
         <origin xyz="0 0 ${distance_shoulder_arm_z}" rpy="${PI/2} ${-PI/2} 0" />
-		<limit effort="1" velocity="1.0" lower="${limit_low_arm_rotation}" upper="${limit_up_arm_rotation}" />
-		<axis xyz="0 0 1" />
-	</joint>
-	<joint name="joint_3" type="revolute">
+          <limit effort="1" velocity="1.0" lower="${limit_low_arm_rotation}" upper="${limit_up_arm_rotation}" />
+          <axis xyz="0 0 1" />
+    </joint>
+    <joint name="joint_3" type="revolute">
         <parent link="arm_link" />
         <child link="elbow_link" />
         <origin xyz="${distance_arm_elbow_x} ${distance_arm_elbow_y} 0" rpy="0 0 ${-PI/2}" />
-		<limit effort="1" velocity="1.0" lower="${limit_low_elbow_rotation}" upper="${limit_up_elbow_rotation}" />
-		<axis xyz="0 0 1" />
-	</joint>
-	<joint name="joint_4" type="revolute">
+          <limit effort="1" velocity="1.0" lower="${limit_low_elbow_rotation}" upper="${limit_up_elbow_rotation}" />
+          <axis xyz="0 0 1" />
+    </joint>
+    <joint name="joint_4" type="revolute">
         <parent link="elbow_link" />
         <child link="forearm_link" />
         <origin xyz="${distance_elbow_forearm_x} ${distance_elbow_forearm_y} 0" rpy="0 ${PI/2} 0" />
-		<limit effort="1" velocity="1.0" lower="${limit_low_forearm_rotation}" upper="${limit_up_forearm_rotation}" />
-		<axis xyz="0 0 1" />
-	</joint>
-	<joint name="joint_5" type="revolute">
+          <limit effort="1" velocity="1.0" lower="${limit_low_forearm_rotation}" upper="${limit_up_forearm_rotation}" />
+          <axis xyz="0 0 1" />
+    </joint>
+    <joint name="joint_5" type="revolute">
         <parent link="forearm_link" />
         <child link="wrist_link" />
-		<origin xyz="0 0 ${distance_forearm_wrist_z}" rpy="0 ${-PI/2} 0" />
-		<limit effort="1" velocity="1.0" lower="${limit_low_wrist_rotation}" upper="${limit_up_wrist_rotation}" />
-		<axis xyz="0 0 1" />
-	</joint>
-	<joint name="joint_6" type="revolute">
+          <origin xyz="0 0 ${distance_forearm_wrist_z}" rpy="0 ${-PI/2} 0" />
+          <limit effort="1" velocity="1.0" lower="${limit_low_wrist_rotation}" upper="${limit_up_wrist_rotation}" />
+          <axis xyz="0 0 1" />
+    </joint>
+    <joint name="joint_6" type="revolute">
         <parent link="wrist_link" />
         <child link="hand_link" />
         <origin xyz="${distance_wrist_hand_x} ${distance_wrist_hand_y} 0" rpy="0 ${PI/2} 0" />
-		<limit effort="1" velocity="1.0" lower="${limit_low_hand_rotation}" upper="${limit_up_hand_rotation}" />
-		<axis xyz="0 0 1" />
-	</joint>
+          <limit effort="1" velocity="1.0" lower="${limit_low_hand_rotation}" upper="${limit_up_hand_rotation}" />
+          <axis xyz="0 0 1" />
+    </joint>
 	<joint name="hand_tool_joint" type="fixed">
         <parent link="hand_link" />

File: niryo_one_description/urdf/v2/niryo_one.urdf.xacro (robot description, xacro)
@@ -40,4 +40,7 @@
     <xacro:property name="limit_low_hand_rotation" value="-2.57436" />
     <xacro:property name="limit_up_hand_rotation" value="2.57436" />
+    <xacro:include filename="$(find niryo_one_description)/urdf/gazebo/niryo_one_v2.gazebo.xacro" />
+	<xacro:include filename="$(find niryo_one_description)/urdf/gazebo/utils.xacro" />
+	<xacro:include filename="$(find niryo_one_description)/urdf/gazebo/niryo_one.transmission.xacro" />
 	<!-- Links -->
     <link name="ground_link"/>
@@ -55,4 +58,13 @@
             </geometry>
         </collision>
+        <inertial>
+      		<origin xyz="0 0 0" rpy="0 0 0"/>
+      		<mass value="2"/>
+			<!--to change-->
+      		<inertia
+        		ixx="0.0" ixy="0.0" ixz="0.0"
+        		iyy="0.0" iyz="0.0"
+        		izz="0.0"/>
+    	</inertial>
 	</link>
     <link name="shoulder_link">
@@ -69,4 +81,12 @@
             </geometry>
         </collision>
+        <inertial>
+      		<origin xyz="0 0 0" rpy="0 0 0"/>
+      		<mass value="1"/>
+      		<inertia
+        		ixx="1.0" ixy="0.0" ixz="0.0"
+        		iyy="1.0" iyz="0.0"
+        		izz="1.0"/>
+    	</inertial>
 	</link>
     <link name="arm_link">
@@ -83,4 +103,12 @@
             </geometry>
         </collision>
+        <inertial>
+      		<origin xyz="0 0 0" rpy="0 0 0"/>
+      		<mass value="0.5"/>
+      		<inertia
+        		ixx="1.0" ixy="0.0" ixz="0.0"
+        		iyy="1.0" iyz="0.0"
+        		izz="1.0"/>
+    	</inertial>
 	</link>
     <link name="elbow_link">
@@ -97,4 +125,12 @@
             </geometry>
         </collision>
+        <inertial>
+      		<origin xyz="0 0 0" rpy="0 0 0"/>
+      		<mass value="0.4"/>
+      		<inertia
+        		ixx="1.0" ixy="0.0" ixz="0.0"
+        		iyy="1.0" iyz="0.0"
+        		izz="1.0"/>
+    	</inertial>
 	</link>
     <link name="forearm_link">
@@ -111,4 +147,12 @@
             </geometry>
         </collision>
+        <inertial>
+      		<origin xyz="0 0 0" rpy="0 0 0"/>
+      		<mass value="0.3"/>
+      		<inertia
+        		ixx="1.0" ixy="0.0" ixz="0.0"
+        		iyy="1.0" iyz="0.0"
+        		izz="1.0"/>
+    	</inertial>
 	</link>
     <link name="wrist_link">
@@ -125,4 +169,12 @@
             </geometry>
         </collision>
+        <inertial>
+      		<origin xyz="0 0 0" rpy="0 0 0"/>
+      		<mass value="0.2"/>
+      		<inertia
+        		ixx="1.0" ixy="0.0" ixz="0.0"
+        		iyy="1.0" iyz="0.0"
+        		izz="1.0"/>
+    	</inertial>
 	</link>
     <link name="hand_link">
@@ -139,4 +191,12 @@
             </geometry>
         </collision>
+        <inertial>
+      		<origin xyz="0 0 0" rpy="0 0 0"/>
+      		<mass value="0.1"/>
+      		<inertia
+        		ixx="1.0" ixy="0.0" ixz="0.0"
+        		iyy="1.0" iyz="0.0"
+        		izz="1.0"/>
+    	</inertial>
 	</link>
     <link name="tool_link">
@@ -195,3 +255,8 @@
         <origin xyz="0 0 ${distance_hand_tool}" rpy="${-PI/2} ${-PI/2} 0" />
 	</joint>
+    <!--plugin-->
+	<gazebo>
+  		<plugin name="gazebo_ros_control" filename="libgazebo_ros_control.so">
+  		</plugin>
+  	</gazebo>
 </robot>

Commit message: Rename 'ground_link' to 'world'

File: niryo_one_description/urdf/v1/niryo_one.urdf.xacro (robot description, xacro)
@@ -41,5 +41,5 @@
     <xacro:property name="limit_up_hand_rotation" value="2.57" />
 	<!-- Links -->
-    <link name="ground_link"/>
+    <link name="world"/>
     <link name="base_link">
 		<visual>
@@ -165,6 +165,6 @@
 	</link>
 	<!--Joints -->
-    <joint name="ground_joint" type="fixed">
-        <parent link="ground_link" />
+    <joint name="joint_world" type="fixed">
+        <parent link="world" />
         <child link="base_link" />
         <origin xyz="0 0 0" rpy="0 0 0" />

File: niryo_one_description/urdf/v1/without_mesh_niryo_one.urdf.xacro (robot description, xacro)
@@ -41,5 +41,5 @@
     <xacro:property name="limit_up_hand_rotation" value="2.57" />
 	<!-- Links -->
-    <link name="ground_link"/>
+    <link name="world"/>
     <link name="base_link">
 	</link>
@@ -59,6 +59,6 @@
 	</link>
 	<!--Joints -->
-    <joint name="ground_joint" type="fixed">
-        <parent link="ground_link" />
+    <joint name="joint_world" type="fixed">
+        <parent link="world" />
         <child link="base_link" />
         <origin xyz="0 0 0" rpy="0 0 0" />

File: niryo_one_description/urdf/v2/niryo_one.urdf.xacro (robot description, xacro)
@@ -41,5 +41,5 @@
     <xacro:property name="limit_up_hand_rotation" value="2.57436" />
 	<!-- Links -->
-    <link name="ground_link"/>
+    <link name="world"/>
     <link name="base_link">
 		<visual>
@@ -143,6 +143,6 @@
 	</link>
 	<!--Joints -->
-    <joint name="ground_joint" type="fixed">
-        <parent link="ground_link" />
+    <joint name="joint_world" type="fixed">
+        <parent link="world" />
         <child link="base_link" />
         <origin xyz="0 0 0" rpy="0 0 0" />

File: niryo_one_description/urdf/v2/without_mesh_niryo_one.urdf.xacro (robot description, xacro)
@@ -41,5 +41,5 @@
     <xacro:property name="limit_up_hand_rotation" value="2.57436" />
 	<!-- Links -->
-    <link name="ground_link"/>
+    <link name="world"/>
     <link name="base_link">
 	</link>
@@ -59,6 +59,6 @@
 	</link>
 	<!--Joints -->
-    <joint name="ground_joint" type="fixed">
-        <parent link="ground_link" />
+    <joint name="joint_world" type="fixed">
+        <parent link="world" />
         <child link="base_link" />
         <origin xyz="0 0 0" rpy="0 0 0" />
