Commit message: organize xacro gazebo files

File: niryo_one_description/urdf/gazebo_utils/niryo_one.gazebo.xacro (robot description, xacro)
@@ -1,3 +1,18 @@
 <?xml version="1.0"?>
+<!--
+    niryo_one.urdf.xacro
+    Copyright (C) 2018 Niryo
+    All rights reserved.
+    This program is free software: you can redistribute it and/or modify
+    it under the terms of the GNU General Public License as published by
+    the Free Software Foundation, either version 3 of the License, or
+    (at your option) any later version.
+    This program is distributed in the hope that it will be useful,
+    but WITHOUT ANY WARRANTY; without even the implied warranty of
+    MERCHANTABILITY or FITNESS FOR A PARTICULAR PURPOSE.  See the
+    GNU General Public License for more details.
+    You should have received a copy of the GNU General Public License
+    along with this program.  If not, see <http://www.gnu.org/licenses/
+-->
 <robot xmlns:xacro="http://www.ros.org/wiki/xacro" name="niryo_one">
   <gazebo reference="ground_link">
@@ -11,42 +26,28 @@
   <gazebo reference="shoulder_link">
 		<material>Gazebo/Black</material>
-		  <mu1>0.0</mu1>
-  		<mu2>0.0</mu2>
 		<turnGravityOff>true</turnGravityOff>
 	</gazebo>
   <gazebo reference="arm_link">
 		<material>Gazebo/Blue</material>
-		<mu1>0.0</mu1>
-  	<mu2>0.0</mu2>
 		<turnGravityOff>true</turnGravityOff>
 	</gazebo>
   <gazebo reference="elbow_link">
 		<material>Gazebo/Black</material>
-		<mu1>0.0</mu1>
-  	<mu2>0.0</mu2>
 		<turnGravityOff>true</turnGravityOff>
 	</gazebo>
   <gazebo reference="forearm_link">
 		<material>Gazebo/Blue</material>
-		<mu1>0.0</mu1>
-  	<mu2>0.0</mu2>
 		<turnGravityOff>true</turnGravityOff>
 	</gazebo>
   <gazebo reference="wrist_link">
 		<material>Gazebo/Black</material>
-		<mu1>0.0</mu1>
-  	<mu2>0.0</mu2>
 		<turnGravityOff>true</turnGravityOff>
 	</gazebo>
   <gazebo reference="hand_link">
 		<material>Gazebo/Blue</material>
-		<mu1>0.0</mu1>
-  	<mu2>0.0</mu2>
 		<turnGravityOff>true</turnGravityOff>
 	</gazebo>
 	<gazebo reference="gripper_link">
 		<material>Gazebo/Black</material>
-		<mu1>0.0</mu1>
-  	<mu2>0.0</mu2>
 		<turnGravityOff>true</turnGravityOff>
 	</gazebo>

File: niryo_one_description/urdf/v1/niryo_one.urdf.xacro (robot description, xacro)
@@ -43,5 +43,7 @@
     <xacro:property name="limit_low_hand_rotation" value="-2.57" />
     <xacro:property name="limit_up_hand_rotation" value="2.57" />
-    <xacro:include filename="$(find niryo_one_description)/urdf/v1/niryo_one.gazebo.xacro" />
+    <xacro:include filename="$(find niryo_one_description)/urdf/gazebo_utils/niryo_one.gazebo.xacro" />
+	<xacro:include filename="$(find niryo_one_description)/urdf/gazebo_utils/utils.xacro" />
+	<xacro:include filename="$(find niryo_one_description)/urdf/gazebo_utils/niryo_one.transmission.xacro" />
 	<!-- Links -->
     <link name="ground_link"/>
@@ -65,4 +67,5 @@
       		<origin xyz="0 0 0" rpy="0 0 0"/>
       		<mass value="1.3"/>
+			<!--to change-->
       		<inertia
         		ixx="0.0" ixy="0.0" ixz="0.0"
@@ -225,5 +228,5 @@
 	</link>
 	<!--Joints -->
-    <joint name="ground_joint" type="fixed">
+	<joint name="ground_joint" type="fixed">
         <parent link="ground_link" />
         <child link="base_link" />
@@ -277,62 +280,4 @@
         <origin xyz="0 0 ${distance_hand_gripper}" rpy="${-PI/2} ${-PI/2} 0" />
 	</joint>
-	<!--transmission-->
-	<transmission name="base_shoulder_transmission">
-      <type>transmission_interface/SimpleTransmission</type>
-      <joint name="joint_1">
-        <hardwareInterface>hardware_interface/PositionJointInterface</hardwareInterface>
-      </joint>
-      <actuator name="base_shoulder_motor">
-        <mechanicalReduction>1</mechanicalReduction>
-		<hardwareInterface>hardware_interface/PositionJointInterface</hardwareInterface>
-      </actuator>
-    </transmission>
-	<transmission name="shoulder_arm_transmission">
-      <type>transmission_interface/SimpleTransmission</type>
-      <joint name="joint_2">
-        <hardwareInterface>hardware_interface/PositionJointInterface</hardwareInterface>
-      </joint>
-      <actuator name="shoulder_arm_motor">
-        <mechanicalReduction>1</mechanicalReduction>
-		<hardwareInterface>hardware_interface/PositionJointInterface</hardwareInterface>
-      </actuator>
-    </transmission>
-	<transmission name="arm_elbow_transmission">
-      <type>transmission_interface/SimpleTransmission</type>
-      <joint name="joint_3">
-        <hardwareInterface>hardware_interface/PositionJointInterface</hardwareInterface>
-      </joint>
-      <actuator name="arm_elbow_motor">
-        <mechanicalReduction>1</mechanicalReduction>
-		<hardwareInterface>hardware_interface/PositionJointInterface</hardwareInterface>
-      </actuator>
-    </transmission>
-	<transmission name="elbow_forarm_transmission">
-      <type>transmission_interface/SimpleTransmission</type>
-      <joint name="joint_4">
-        <hardwareInterface>hardware_interface/PositionJointInterface</hardwareInterface>
-      </joint>
-      <actuator name="elbow_forarm_motor">
-        <mechanicalReduction>1</mechanicalReduction>
-      </actuator>
-    </transmission>
-	<transmission name="forarm_wirst_transmission">
-      <type>transmission_interface/SimpleTransmission</type>
-      <joint name="joint_5">
-        <hardwareInterface>hardware_interface/PositionJointInterface</hardwareInterface>
-      </joint>
-      <actuator name="forarm_wirst_motor">
-        <mechanicalReduction>1</mechanicalReduction>
-      </actuator>
-    </transmission>
-	<transmission name="wirst_gripper_transmission">
-      <type>transmission_interface/SimpleTransmission</type>
-      <joint name="joint_6">
-        <hardwareInterface>hardware_interface/PositionJointInterface</hardwareInterface>
-      </joint>
-      <actuator name="wirst_gripper_motor">
-        <mechanicalReduction>1</mechanicalReduction>
-      </actuator>
-    </transmission>
 	<!--plugin-->
 	<gazebo>

Commit message: include niryo_one_base in niryo_one_gazebo.launch

File: niryo_one_description/urdf/gazebo_utils/niryo_one.gazebo.xacro (robot description, xacro)
@@ -17,5 +17,5 @@
 <robot xmlns:xacro="http://www.ros.org/wiki/xacro" name="niryo_one">
   <gazebo reference="ground_link">
-		<material>Gazebo/Blue</material>
+		<material>Gazebo/Back</material>
 		<turnGravityOff>true</turnGravityOff>
 	</gazebo>

File: niryo_one_description/urdf/v1/niryo_one.urdf.xacro (robot description, xacro)
@@ -47,5 +47,5 @@
 	<xacro:include filename="$(find niryo_one_description)/urdf/gazebo_utils/niryo_one.transmission.xacro" />
 	<!-- Links -->
-    <link name="ground_link"/>
+	<link name="ground_link"/>
     <link name="base_link">
 		<visual>
@@ -231,5 +231,5 @@
         <parent link="ground_link" />
         <child link="base_link" />
-        <origin xyz="0 0 0" rpy="0 0 0" />
+        <origin xyz="0.0 0.0 0.0" rpy="0 0 0" />
     </joint>
 	<joint name="joint_1" type="revolute">
