Commit message: add hardware version v2 to gazebo simulation

File: niryo_one_description/urdf/gazebo/niryo_one.gazebo.xacro (robot description, xacro)
@@ -17,5 +17,5 @@
 <robot xmlns:xacro="http://www.ros.org/wiki/xacro" name="niryo_one">
   <gazebo reference="ground_link">
-		<material>Gazebo/Back</material>
+		<material>Gazebo/Black</material>
 		<turnGravityOff>true</turnGravityOff>
 	</gazebo>

File: niryo_one_description/urdf/gazebo/niryo_one.transmission.xacro (robot description, xacro)
@@ -22,6 +22,6 @@
         <hardwareInterface>hardware_interface/PositionJointInterface</hardwareInterface>
       </joint>
-      <actuator name="base_shoulder_motor">
-        <mechanicalReduction>1</mechanicalReduction>
+      <actuator name="base_shoulder_stepper">
+        <mechanicalReduction>6.0625</mechanicalReduction>
 		<hardwareInterface>hardware_interface/PositionJointInterface</hardwareInterface>
       </actuator>
@@ -32,6 +32,6 @@
         <hardwareInterface>hardware_interface/PositionJointInterface</hardwareInterface>
       </joint>
-      <actuator name="shoulder_arm_motor">
-        <mechanicalReduction>1</mechanicalReduction>
+      <actuator name="shoulder_arm_stepper">
+        <mechanicalReduction>8.3125</mechanicalReduction>
 		<hardwareInterface>hardware_interface/PositionJointInterface</hardwareInterface>
       </actuator>
@@ -42,6 +42,6 @@
         <hardwareInterface>hardware_interface/PositionJointInterface</hardwareInterface>
       </joint>
-      <actuator name="arm_elbow_motor">
-        <mechanicalReduction>1</mechanicalReduction>
+      <actuator name="arm_elbow_stepper">
+        <mechanicalReduction>7.875</mechanicalReduction>
 		<hardwareInterface>hardware_interface/PositionJointInterface</hardwareInterface>
       </actuator>
@@ -53,5 +53,5 @@
       </joint>
       <actuator name="elbow_forarm_motor">
-        <mechanicalReduction>1</mechanicalReduction>
+        <mechanicalReduction>5.0</mechanicalReduction>
       </actuator>
     </transmission>

File: niryo_one_description/urdf/v1/niryo_one.urdf.xacro (robot description, xacro)
@@ -43,7 +43,7 @@
     <xacro:property name="limit_low_hand_rotation" value="-2.57" />
     <xacro:property name="limit_up_hand_rotation" value="2.57" />
-    <xacro:include filename="$(find niryo_one_description)/urdf/gazebo_utils/niryo_one.gazebo.xacro" />
-	<xacro:include filename="$(find niryo_one_description)/urdf/gazebo_utils/utils.xacro" />
-	<xacro:include filename="$(find niryo_one_description)/urdf/gazebo_utils/niryo_one.transmission.xacro" />
+    <xacro:include filename="$(find niryo_one_description)/urdf/gazebo/niryo_one.gazebo.xacro" />
+	<xacro:include filename="$(find niryo_one_description)/urdf/gazebo/utils.xacro" />
+	<xacro:include filename="$(find niryo_one_description)/urdf/gazebo/niryo_one.transmission.xacro" />
 	<!-- Links -->
 	<link name="ground_link"/>

File: niryo_one_description/urdf/v2/niryo_one.urdf.xacro (robot description, xacro)
@@ -45,4 +45,7 @@
     <xacro:property name="limit_low_hand_rotation" value="-2.57" />
     <xacro:property name="limit_up_hand_rotation" value="2.57" />
+    <xacro:include filename="$(find niryo_one_description)/urdf/gazebo/niryo_one.gazebo.xacro" />
+	<xacro:include filename="$(find niryo_one_description)/urdf/gazebo/utils.xacro" />
+	<xacro:include filename="$(find niryo_one_description)/urdf/gazebo/niryo_one.transmission.xacro" />
 	<!-- Links -->
     <link name="ground_link"/>
@@ -63,4 +66,13 @@
             </geometry>
         </collision>
+        <inertial>
+      		<origin xyz="0 0 0" rpy="0 0 0"/>
+      		<mass value="1.3"/>
+			<!--to change-->
+      		<inertia
+        		ixx="0.0" ixy="0.0" ixz="0.0"
+        		iyy="0.0" iyz="0.0"
+        		izz="0.0"/>
+    	</inertial>
 	</link>
     <link name="shoulder_link">
@@ -80,4 +92,12 @@
             </geometry>
         </collision>
+        <inertial>
+      		<origin xyz="0 0 0" rpy="0 0 0"/>
+      		<mass value="0.6"/>
+      		<inertia
+        		ixx="1.0" ixy="0.0" ixz="0.0"
+        		iyy="1.0" iyz="0.0"
+        		izz="1.0"/>
+    	</inertial>
 	</link>
     <link name="arm_link">
@@ -97,4 +117,12 @@
             </geometry>
         </collision>
+        <inertial>
+      		<origin xyz="0 0 0" rpy="0 0 0"/>
+      		<mass value="0.5"/>
+      		<inertia
+        		ixx="1.0" ixy="0.0" ixz="0.0"
+        		iyy="1.0" iyz="0.0"
+        		izz="1.0"/>
+    	</inertial>
 	</link>
     <link name="elbow_link">
@@ -115,4 +143,12 @@
             </geometry>
         </collision>
+        <inertial>
+      		<origin xyz="0 0 0" rpy="0 0 0"/>
+      		<mass value="0.4"/>
+      		<inertia
+        		ixx="1.0" ixy="0.0" ixz="0.0"
+        		iyy="1.0" iyz="0.0"
+        		izz="1.0"/>
+    	</inertial>
 	</link>
     <link name="forearm_link">
@@ -132,4 +168,12 @@
             </geometry>
         </collision>
+        <inertial>
+      		<origin xyz="0 0 0" rpy="0 0 0"/>
+      		<mass value="0.3"/>
+      		<inertia
+        		ixx="1.0" ixy="0.0" ixz="0.0"
+        		iyy="1.0" iyz="0.0"
+        		izz="1.0"/>
+    	</inertial>
 	</link>
     <link name="wrist_link">
@@ -149,4 +193,12 @@
             </geometry>
         </collision>
+        <inertial>
+      		<origin xyz="0 0 0" rpy="0 0 0"/>
+      		<mass value="0.2"/>
+      		<inertia
+        		ixx="1.0" ixy="0.0" ixz="0.0"
+        		iyy="1.0" iyz="0.0"
+        		izz="1.0"/>
+    	</inertial>
 	</link>
     <link name="hand_link">
@@ -166,4 +218,12 @@
             </geometry>
         </collision>
+        <inertial>
+      		<origin xyz="0 0 0" rpy="0 0 0"/>
+      		<mass value="0.1"/>
+      		<inertia
+        		ixx="1.0" ixy="0.0" ixz="0.0"
+        		iyy="1.0" iyz="0.0"
+        		izz="1.0"/>
+    	</inertial>
 	</link>
     <link name="gripper_link">
@@ -222,3 +282,8 @@
         <origin xyz="0 0 ${distance_hand_gripper}" rpy="${-PI/2} ${-PI/2} 0" />
 	</joint>
+    <!--plugin-->
+	<gazebo>
+  		<plugin name="gazebo_ros_control" filename="libgazebo_ros_control.so">
+  		</plugin>
+  	</gazebo>
 </robot>

Commit message: add gazebo xacro model description

File: niryo_one_description/urdf/gazebo/niryo_one.gazebo.xacro (robot description, xacro)
@@ -17,38 +17,37 @@
 <robot xmlns:xacro="http://www.ros.org/wiki/xacro" name="niryo_one">
   <gazebo reference="ground_link">
-		<material>Gazebo/Black</material>
-		<turnGravityOff>true</turnGravityOff>
-	</gazebo>
+        <turnGravityOff>true</turnGravityOff>
+     </gazebo>
   <gazebo reference="base_link">
-		<material>>Gazebo/Black</material>
-		<turnGravityOff>true</turnGravityOff>
-	</gazebo>
+          <material>>Gazebo/Black</material>
+          <turnGravityOff>true</turnGravityOff>
+     </gazebo>
   <gazebo reference="shoulder_link">
-		<material>Gazebo/Black</material>
-		<turnGravityOff>true</turnGravityOff>
-	</gazebo>
+          <material>Gazebo/Black</material>
+          <turnGravityOff>true</turnGravityOff>
+     </gazebo>
   <gazebo reference="arm_link">
-		<material>Gazebo/Blue</material>
-		<turnGravityOff>true</turnGravityOff>
-	</gazebo>
+          <material>Gazebo/Blue</material>
+          <turnGravityOff>true</turnGravityOff>
+     </gazebo>
   <gazebo reference="elbow_link">
-		<material>Gazebo/Black</material>
-		<turnGravityOff>true</turnGravityOff>
-	</gazebo>
+          <material>Gazebo/Black</material>
+          <turnGravityOff>true</turnGravityOff>
+     </gazebo>
   <gazebo reference="forearm_link">
-		<material>Gazebo/Blue</material>
-		<turnGravityOff>true</turnGravityOff>
-	</gazebo>
+          <material>Gazebo/Blue</material>
+          <turnGravityOff>true</turnGravityOff>
+     </gazebo>
   <gazebo reference="wrist_link">
-		<material>Gazebo/Black</material>
-		<turnGravityOff>true</turnGravityOff>
-	</gazebo>
+          <material>Gazebo/Black</material>
+          <turnGravityOff>true</turnGravityOff>
+     </gazebo>
   <gazebo reference="hand_link">
-		<material>Gazebo/Blue</material>
-		<turnGravityOff>true</turnGravityOff>
-	</gazebo>
-	<gazebo reference="gripper_link">
-		<material>Gazebo/Black</material>
-		<turnGravityOff>true</turnGravityOff>
-	</gazebo>
+          <material>Gazebo/Blue</material>
+          <turnGravityOff>true</turnGravityOff>
+     </gazebo>
+     <gazebo reference="gripper_link">
+          <material>Gazebo/Black</material>
+          <turnGravityOff>true</turnGravityOff>
+     </gazebo>
 </robot>

File: niryo_one_description/urdf/gazebo/niryo_one.transmission.xacro (robot description, xacro)
@@ -16,6 +16,6 @@
 -->
 <robot xmlns:xacro="http://www.ros.org/wiki/xacro" name="niryo_one">
-	<!--transmission-->
-	<transmission name="base_shoulder_transmission">
+     <!--transmission-->
+     <transmission name="base_shoulder_transmission">
       <type>transmission_interface/SimpleTransmission</type>
       <joint name="joint_1">
@@ -24,8 +24,8 @@
       <actuator name="base_shoulder_stepper">
         <mechanicalReduction>6.0625</mechanicalReduction>
-		<hardwareInterface>hardware_interface/PositionJointInterface</hardwareInterface>
+          <hardwareInterface>hardware_interface/PositionJointInterface</hardwareInterface>
       </actuator>
     </transmission>
-	<transmission name="shoulder_arm_transmission">
+     <transmission name="shoulder_arm_transmission">
       <type>transmission_interface/SimpleTransmission</type>
       <joint name="joint_2">
@@ -34,8 +34,8 @@
       <actuator name="shoulder_arm_stepper">
         <mechanicalReduction>8.3125</mechanicalReduction>
-		<hardwareInterface>hardware_interface/PositionJointInterface</hardwareInterface>
+          <hardwareInterface>hardware_interface/PositionJointInterface</hardwareInterface>
       </actuator>
     </transmission>
-	<transmission name="arm_elbow_transmission">
+     <transmission name="arm_elbow_transmission">
       <type>transmission_interface/SimpleTransmission</type>
       <joint name="joint_3">
@@ -44,8 +44,8 @@
       <actuator name="arm_elbow_stepper">
         <mechanicalReduction>7.875</mechanicalReduction>
-		<hardwareInterface>hardware_interface/PositionJointInterface</hardwareInterface>
+          <hardwareInterface>hardware_interface/PositionJointInterface</hardwareInterface>
       </actuator>
     </transmission>
-	<transmission name="elbow_forarm_transmission">
+     <transmission name="elbow_forarm_transmission">
       <type>transmission_interface/SimpleTransmission</type>
       <joint name="joint_4">
@@ -56,5 +56,5 @@
       </actuator>
     </transmission>
-	<transmission name="forarm_wirst_transmission">
+     <transmission name="forarm_wirst_transmission">
       <type>transmission_interface/SimpleTransmission</type>
       <joint name="joint_5">
@@ -65,5 +65,5 @@
       </actuator>
     </transmission>
-	<transmission name="wirst_gripper_transmission">
+     <transmission name="wirst_gripper_transmission">
       <type>transmission_interface/SimpleTransmission</type>
       <joint name="joint_6">

File: niryo_one_description/urdf/gazebo/utils.xacro (robot description, xacro)
@@ -2,16 +2,18 @@
 <robot xmlns:xacro="http://www.ros.org/wiki/xacro">
   <!-- Little helper macro to define the inertia matrix needed for links. -->
-  <xacro:macro name="cuboid_inertia_def" params="width height length mass">
-    <inertia ixx="${mass * (height * height + length * length) / 12}"
-             iyy="${mass * (width * width + length * length) / 12}"
-             izz="${mass * (width * width + height * height) / 12}"
-             ixy="0" iyz="0" ixz="0"/>
+  <xacro:macro name="cylinder_inertia" params="m r h">
+    <inertia  ixx="${m*(3*r*r+h*h)/12}" ixy = "0" ixz = "0"
+              iyy="${m*(3*r*r+h*h)/12}" iyz = "0"
+              izz="${m*r*r/2}" />
   </xacro:macro>
-  <!-- length is along the y-axis! -->
-  <xacro:macro name="cylinder_inertia_def" params="radius length mass">
-    <inertia ixx="${mass * (3 * radius * radius + length * length) / 12}"
-             iyy="${mass * radius* radius / 2}"
-             izz="${mass * (3 * radius * radius + length * length) / 12}"
-             ixy="0" iyz="0" ixz="0"/>
+  <xacro:macro name="box_inertia" params="m x y z">
+    <inertia  ixx="${m*(y*y+z*z)/12}" ixy = "0" ixz = "0"
+              yy="${m*(x*x+z*z)/12}" iyz = "0"
+              izz="${m*(x*x+z*z)/12}" />
   </xacro:macro>
+  <xacro:macro name="sphere_inertia" params="m r">
+    <inertia  ixx="${2*m*r*r/5}" ixy = "0" ixz = "0"
+              iyy="${2*m*r*r/5}" iyz = "0"
+              izz="${2*m*r*r/5}" />
+    </xacro:macro>
 </robot>

Commit message: comment gazebo colors to use stl colors

File: niryo_one_description/urdf/gazebo/niryo_one.gazebo.xacro (robot description, xacro)
@@ -20,33 +20,33 @@
      </gazebo>
   <gazebo reference="base_link">
-          <material>>Gazebo/Black</material>
+          <!-- <material>>Gazebo/Black</material> -->
           <turnGravityOff>true</turnGravityOff>
      </gazebo>
   <gazebo reference="shoulder_link">
-          <material>Gazebo/Black</material>
+          <!-- <material>Gazebo/Black</material> -->
           <turnGravityOff>true</turnGravityOff>
      </gazebo>
   <gazebo reference="arm_link">
-          <material>Gazebo/Blue</material>
+          <!-- <material>Gazebo/Blue</material> -->
           <turnGravityOff>true</turnGravityOff>
      </gazebo>
   <gazebo reference="elbow_link">
-          <material>Gazebo/Black</material>
+          <!-- <material>Gazebo/Black</material> -->
           <turnGravityOff>true</turnGravityOff>
      </gazebo>
   <gazebo reference="forearm_link">
-          <material>Gazebo/Blue</material>
+          <!-- <material>Gazebo/Blue</material> -->
           <turnGravityOff>true</turnGravityOff>
      </gazebo>
   <gazebo reference="wrist_link">
-          <material>Gazebo/Black</material>
+          <!-- <material>Gazebo/Black</material> -->
           <turnGravityOff>true</turnGravityOff>
      </gazebo>
   <gazebo reference="hand_link">
-          <material>Gazebo/Blue</material>
+          <!-- <material>Gazebo/Blue</material> -->
           <turnGravityOff>true</turnGravityOff>
      </gazebo>
-     <gazebo reference="gripper_link">
-          <material>Gazebo/Black</material>
+     <gazebo reference="tool_link">
+          <!-- <material>Gazebo/Black</material> -->
           <turnGravityOff>true</turnGravityOff>
      </gazebo>

Commit message: restore niryo_one V1 colors

File: niryo_one_description/urdf/gazebo/niryo_one.gazebo.xacro (robot description, xacro)
@@ -20,33 +20,33 @@
      </gazebo>
   <gazebo reference="base_link">
-          <!-- <material>>Gazebo/Black</material> -->
+          <material>>Gazebo/Black</material>
           <turnGravityOff>true</turnGravityOff>
      </gazebo>
   <gazebo reference="shoulder_link">
-          <!-- <material>Gazebo/Black</material> -->
+          <material>Gazebo/Black</material>
           <turnGravityOff>true</turnGravityOff>
      </gazebo>
   <gazebo reference="arm_link">
-          <!-- <material>Gazebo/Blue</material> -->
+          <material>Gazebo/Blue</material>
           <turnGravityOff>true</turnGravityOff>
      </gazebo>
   <gazebo reference="elbow_link">
-          <!-- <material>Gazebo/Black</material> -->
+          <material>Gazebo/Black</material>
           <turnGravityOff>true</turnGravityOff>
      </gazebo>
   <gazebo reference="forearm_link">
-          <!-- <material>Gazebo/Blue</material> -->
+          <material>Gazebo/Blue</material>
           <turnGravityOff>true</turnGravityOff>
      </gazebo>
   <gazebo reference="wrist_link">
-          <!-- <material>Gazebo/Black</material> -->
+          <material>Gazebo/Black</material>
           <turnGravityOff>true</turnGravityOff>
      </gazebo>
   <gazebo reference="hand_link">
-          <!-- <material>Gazebo/Blue</material> -->
+          <material>Gazebo/Blue</material>
           <turnGravityOff>true</turnGravityOff>
      </gazebo>
      <gazebo reference="tool_link">
-          <!-- <material>Gazebo/Black</material> -->
+          <material>Gazebo/Black</material>
           <turnGravityOff>true</turnGravityOff>
      </gazebo>
