Commit message: update gazebo simulation with ros melodic

File: niryo_one_description/urdf/gazebo/niryo_one_v2.gazebo.xacro (robot description, xacro)
@@ -17,36 +17,28 @@
 <robot xmlns:xacro="http://www.ros.org/wiki/xacro" name="niryo_one">
   <gazebo reference="ground_link">
-        <turnGravityOff>true</turnGravityOff>
+        <turnGravityOff>false</turnGravityOff>
      </gazebo>
   <gazebo reference="base_link">
-          <material>>Gazebo/Black</material>
-          <turnGravityOff>true</turnGravityOff>
+          <turnGravityOff>false</turnGravityOff>
      </gazebo>
   <gazebo reference="shoulder_link">
-          <material>Gazebo/Black</material>
           <turnGravityOff>true</turnGravityOff>
      </gazebo>
   <gazebo reference="arm_link">
-          <material>Gazebo/Blue</material>
           <turnGravityOff>true</turnGravityOff>
      </gazebo>
   <gazebo reference="elbow_link">
-          <material>Gazebo/Black</material>
           <turnGravityOff>true</turnGravityOff>
      </gazebo>
   <gazebo reference="forearm_link">
-          <material>Gazebo/Blue</material>
           <turnGravityOff>true</turnGravityOff>
      </gazebo>
   <gazebo reference="wrist_link">
-          <material>Gazebo/Black</material>
           <turnGravityOff>true</turnGravityOff>
      </gazebo>
   <gazebo reference="hand_link">
-          <material>Gazebo/Blue</material>
           <turnGravityOff>true</turnGravityOff>
      </gazebo>
      <gazebo reference="tool_link">
-          <material>Gazebo/Black</material>
           <turnGravityOff>true</turnGravityOff>
      </gazebo>

File: niryo_one_description/urdf/v1/niryo_one.urdf.xacro (robot description, xacro)
@@ -40,5 +40,5 @@
     <xacro:property name="limit_low_hand_rotation" value="-2.57" />
     <xacro:property name="limit_up_hand_rotation" value="2.57" />
-    <xacro:include filename="$(find niryo_one_description)/urdf/gazebo/niryo_one.gazebo.xacro" />
+    <xacro:include filename="$(find niryo_one_description)/urdf/gazebo/niryo_one_v1.gazebo.xacro" />
     <xacro:include filename="$(find niryo_one_description)/urdf/gazebo/utils.xacro" />
     <xacro:include filename="$(find niryo_one_description)/urdf/gazebo/niryo_one.transmission.xacro" />

File: niryo_one_description/urdf/v2/niryo_one.urdf.xacro (robot description, xacro)
@@ -40,5 +40,5 @@
     <xacro:property name="limit_low_hand_rotation" value="-2.57436" />
     <xacro:property name="limit_up_hand_rotation" value="2.57436" />
-    <xacro:include filename="$(find niryo_one_description)/urdf/gazebo/niryo_one.gazebo.xacro" />
+    <xacro:include filename="$(find niryo_one_description)/urdf/gazebo/niryo_one_v2.gazebo.xacro" />
 	<xacro:include filename="$(find niryo_one_description)/urdf/gazebo/utils.xacro" />
 	<xacro:include filename="$(find niryo_one_description)/urdf/gazebo/niryo_one.transmission.xacro" />
@@ -60,5 +60,5 @@
         <inertial>
       		<origin xyz="0 0 0" rpy="0 0 0"/>
-      		<mass value="1.3"/>
+      		<mass value="2"/>
 			<!--to change-->
       		<inertia
@@ -83,5 +83,5 @@
         <inertial>
       		<origin xyz="0 0 0" rpy="0 0 0"/>
-      		<mass value="0.6"/>
+      		<mass value="1"/>
       		<inertia
         		ixx="1.0" ixy="0.0" ixz="0.0"
