Commit message: refactor some files

File: niryo_one_description/urdf/gazebo/box.urdf.xacro (robot description, xacro)
@@ -1,3 +1,19 @@
-<robot name="simple_box">
+<?xml version="1.0"?>
+<!--
+    niryo_one.urdf.xacro
+    Copyright (C) 2017 Niryo
+    All rights reserved.
+    This program is free software: you can redistribute it and/or modify
+    it under the terms of the GNU General Public License as published by
+    the Free Software Foundation, either version 3 of the License, or
+    (at your option) any later version.
+    This program is distributed in the hope that it will be useful,
+    but WITHOUT ANY WARRANTY; without even the implied warranty of
+    MERCHANTABILITY or FITNESS FOR A PARTICULAR PURPOSE.  See the
+    GNU General Public License for more details.
+    You should have received a copy of the GNU General Public License
+    along with this program.  If not, see <http://www.gnu.org/licenses/>.
+-->
+<robot xmlns:xacro="http://ros.org/wiki/xacro" name="simple_box">
   <link name="box_1">
     <inertial>

File: niryo_one_description/urdf/v1/without_mesh_niryo_one.urdf.xacro (robot description, xacro)
@@ -26,18 +26,8 @@
     <xacro:property name="distance_wrist_hand_x" value="0.018" />
     <xacro:property name="distance_wrist_hand_y" value="0" />
-<<<<<<< HEAD
-    <!-- not yet implemented, tools are handled separately -->
-    <xacro:property name="distance_hand_gripper" value="0.00" />
-    <xacro:property name="thickness_arm_axis" value="0.052" />
-    <xacro:property name="thickness_forearm_axis" value="0.048" />
-    <xacro:property name="PI" value="3.14159265359" />
-    <xacro:property name="limit_low_shoulder_rotation" value="-3.05433" />
-    <xacro:property name="limit_up_shoulder_rotation" value="3.05433" />
-=======
     <xacro:property name="distance_hand_tool" value="0.00" />
 	<xacro:property name="PI" value="3.14159265359" />
 	<xacro:property name="limit_low_shoulder_rotation" value="-3.05433" />
 	<xacro:property name="limit_up_shoulder_rotation" value="3.05433" />
->>>>>>> f9562b7a28424a0d9a25d0dd6343b672fabdfdae
     <xacro:property name="limit_low_arm_rotation" value="${-PI/2}" />
     <xacro:property name="limit_up_arm_rotation" value="0.628319" />
@@ -65,13 +55,7 @@
     </link>
     <link name="hand_link">
-<<<<<<< HEAD
-    </link>
-    <link name="gripper_link">
-    </link>
-=======
 	</link>
     <link name="tool_link">
 	</link>
->>>>>>> f9562b7a28424a0d9a25d0dd6343b672fabdfdae
      <!--Joints -->
     <joint name="ground_joint" type="fixed">
@@ -122,11 +106,4 @@
           <axis xyz="0 0 1" />
     </joint>
-<<<<<<< HEAD
-    <joint name="hand_gripper_joint" type="fixed">
-        <parent link="hand_link" />
-        <child link="gripper_link" />
-        <origin xyz="0 0 ${distance_hand_gripper}" rpy="${-PI/2} ${-PI/2} 0" />
-    </joint>
-=======
 	<joint name="hand_tool_joint" type="fixed">
         <parent link="hand_link" />
@@ -134,4 +111,3 @@
         <origin xyz="0 0 ${distance_hand_tool}" rpy="${-PI/2} ${-PI/2} 0" />
 	</joint>
->>>>>>> f9562b7a28424a0d9a25d0dd6343b672fabdfdae
 </robot>
