Commit message: Update axis 5 limits

File: niryo_one_description/urdf/v2/niryo_one.urdf.xacro (robot description, xacro)
@@ -36,6 +36,6 @@
     <xacro:property name="limit_low_forearm_rotation" value="-3.05433" />
     <xacro:property name="limit_up_forearm_rotation" value="3.05433" />
-    <xacro:property name="limit_low_wrist_rotation" value="-2.0944" />
-    <xacro:property name="limit_up_wrist_rotation" value="2.53073" />
+    <xacro:property name="limit_low_wrist_rotation" value="-1.74533" />
+    <xacro:property name="limit_up_wrist_rotation" value="1.91986" />
     <xacro:property name="limit_low_hand_rotation" value="-2.57436" />
     <xacro:property name="limit_up_hand_rotation" value="2.57436" />

File: niryo_one_description/urdf/v2/without_mesh_niryo_one.urdf.xacro (robot description, xacro)
@@ -36,6 +36,6 @@
     <xacro:property name="limit_low_forearm_rotation" value="-3.05433" />
     <xacro:property name="limit_up_forearm_rotation" value="3.05433" />
-    <xacro:property name="limit_low_wrist_rotation" value="-2.0944" />
-    <xacro:property name="limit_up_wrist_rotation" value="2.53073" />
+    <xacro:property name="limit_low_wrist_rotation" value="-1.74533" />
+    <xacro:property name="limit_up_wrist_rotation" value="1.91986" />
     <xacro:property name="limit_low_hand_rotation" value="-2.57436" />
     <xacro:property name="limit_up_hand_rotation" value="2.57436" />

Commit message: Added 3 Niryo grippers with controller and python script

File: niryo_one_description/urdf/v2/niryo_one.urdf.xacro (robot description, xacro)
@@ -43,4 +43,7 @@
 	<xacro:include filename="$(find niryo_one_description)/urdf/gazebo/utils.xacro" />
 	<xacro:include filename="$(find niryo_one_description)/urdf/gazebo/niryo_one.transmission.xacro" />
+	<!-- Gripper -->
+<!--	<xacro:include filename="$(find niryo_one_description)/urdf/v2/gripper/niryo_gripper_1.urdf.xacro" />  -->
+	<xacro:include filename="$(find niryo_one_description)/urdf/v2/gripper/niryo_gripper_2.urdf.xacro" />
 	<!-- Links -->
     <link name="ground_link"/>
@@ -255,4 +258,11 @@
         <origin xyz="0 0 ${distance_hand_tool}" rpy="${-PI/2} ${-PI/2} 0" />
 	</joint>
+<!--	<xacro:niryo_gripper_1 prefix="gripper_" parent="tool_link" >
+	  <origin xyz="0.025 0 -0.013" rpy="${PI/2} ${PI} ${PI/2} " />
+	</xacro:niryo_gripper_1>
+-->
+	<xacro:niryo_gripper_2 prefix="gripper_" parent="tool_link" >
+	  <origin xyz="0.025 0 -0.013" rpy="${PI/2} ${PI} ${PI/2} " />
+	</xacro:niryo_gripper_2>
     <!--plugin-->
 	<gazebo>

Commit message: Lowering the limit of joint 2

File: niryo_one_description/urdf/v2/niryo_one.urdf.xacro (robot description, xacro)
@@ -30,5 +30,5 @@
     <xacro:property name="limit_low_shoulder_rotation" value="-3.05433" />
     <xacro:property name="limit_up_shoulder_rotation" value="3.05433" />
-    <xacro:property name="limit_low_arm_rotation" value="-1.91986" />
+    <xacro:property name="limit_low_arm_rotation" value="-1.57080" />
     <xacro:property name="limit_up_arm_rotation" value="0.640187" />
     <xacro:property name="limit_low_elbow_rotation" value="-1.397485" />

File: niryo_one_description/urdf/v2/without_mesh_niryo_one.urdf.xacro (robot description, xacro)
@@ -30,5 +30,5 @@
     <xacro:property name="limit_low_shoulder_rotation" value="-3.05433" />
     <xacro:property name="limit_up_shoulder_rotation" value="3.05433" />
-    <xacro:property name="limit_low_arm_rotation" value="-1.91986" />
+    <xacro:property name="limit_low_arm_rotation" value="-1.57080" />
     <xacro:property name="limit_up_arm_rotation" value="0.640187" />
     <xacro:property name="limit_low_elbow_rotation" value="-1.397485" />
