Commit message: working gazebo

File: niryo_one_description/urdf/v2/gazebo_niryo_one.urdf.xacro (robot description, xacro)
@@ -1,3 +1,11 @@
-<?xml version="1.0"?>
+<?xml version="1.0" encoding="utf-8" ?>
+<!-- =================================================================================== -->
+<!-- |    This document was autogenerated by xacro from /home/wolf/ros_ws/src/test_niryo_moveit/n1_description/urdf/gazebo_niryo_one.urdf.xacro | -->
+<!-- |    EDITING THIS FILE BY HAND IS NOT RECOMMENDED                                 | -->
+<!-- =================================================================================== -->
+<!-- =================================================================================== -->
+<!-- |    This document was autogenerated by xacro from /home/wolf/ros_ws/src/test_niryo_moveit/n1_description/urdf/gazebo_niryo_one.urdf.xacro | -->
+<!-- |    EDITING THIS FILE BY HAND IS NOT RECOMMENDED                                 | -->
+<!-- =================================================================================== -->
 <!--
     niryo_one.urdf.xacro
@@ -15,34 +23,11 @@
     along with this program.  If not, see <http://www.gnu.org/licenses/>.
 -->
-<robot xmlns:xacro="http://www.ros.org/wiki/xacro" name="niryo_one">
+<robot name="niryo_one">
     <!-- Properties -->
-    <xacro:property name="distance_origin_shoulder_z" value="0.103" />
-    <xacro:property name="distance_shoulder_arm_z" value="0.080" />
-    <xacro:property name="distance_arm_elbow_x" value="0.210" />
-    <xacro:property name="distance_arm_elbow_y" value="0.0" />
-    <xacro:property name="distance_elbow_forearm_x" value="0.0415" />
-    <xacro:property name="distance_elbow_forearm_y" value="0.030" />
-    <xacro:property name="distance_forearm_wrist_z" value="0.180" />
-    <xacro:property name="distance_wrist_hand_x" value="0.0164" />
-    <xacro:property name="distance_wrist_hand_y" value="-0.0055" />
-    <xacro:property name="distance_hand_tool" value="0.0073" />
-    <xacro:property name="PI" value="3.14159265359" />
-    <xacro:property name="limit_low_shoulder_rotation" value="-3.05433" />
-    <xacro:property name="limit_up_shoulder_rotation" value="3.05433" />
-    <xacro:property name="limit_low_arm_rotation" value="-1.91986" />
-    <xacro:property name="limit_up_arm_rotation" value="0.640187" />
-    <xacro:property name="limit_low_elbow_rotation" value="-1.397485" />
-    <xacro:property name="limit_up_elbow_rotation" value="${PI/2}" />
-    <xacro:property name="limit_low_forearm_rotation" value="-3.05433" />
-    <xacro:property name="limit_up_forearm_rotation" value="3.05433" />
-    <xacro:property name="limit_low_wrist_rotation" value="-1.74533" />
-    <xacro:property name="limit_up_wrist_rotation" value="1.91986" />
-    <xacro:property name="limit_low_hand_rotation" value="-2.57436" />
-    <xacro:property name="limit_up_hand_rotation" value="2.57436" />
     <!-- Links -->
     <link name="world" />
     <link name="base_link">
         <visual>
-            <origin xyz="0 0 0" rpy="0 0 0" />
+            <origin rpy="0 0 0" xyz="0 0 0" />
             <geometry>
                 <mesh filename="package://niryo_one_description/meshes/v2/collada/base_link.dae" />
@@ -50,18 +35,18 @@
         </visual>
         <collision>
-            <origin xyz="0 0 0" rpy="0 0 0" />
+            <origin rpy="0 0 0" xyz="0 0 0" />
             <geometry>
                 <mesh filename="package://niryo_one_description/meshes/v2/stl/base_link.stl" />
             </geometry>
         </collision>
-        <inertial>
-            <origin xyz="0 0 ${distance_origin_shoulder_z / 2}" rpy="0 0 0" />
+<inertial>
+            <origin rpy="0 0 0" xyz="0 0 0.0515" />
             <mass value="1.2" />
-            <inertia ixx="0.0015" ixy="0.0" ixz="0.0" iyy="0.0015" iyz="0.0" izz="0.0015"/>
+            <inertia ixx="0.0015" ixy="0.0" ixz="0.0" iyy="0.0015" iyz="0.0" izz="0.0015" />
         </inertial>
     </link>
     <link name="shoulder_link">
         <visual>
-            <origin xyz="0 0 0" rpy="0 0 0" />
+            <origin rpy="0 0 0" xyz="0 0 0" />
             <geometry>
                 <mesh filename="package://niryo_one_description/meshes/v2/collada/shoulder_link.dae" />
@@ -69,18 +54,18 @@
         </visual>
         <collision>
-            <origin xyz="0 0 0" rpy="0 0 0" />
+            <origin rpy="0 0 0" xyz="0 0 0" />
             <geometry>
                 <mesh filename="package://niryo_one_description/meshes/v2/stl/shoulder_link.stl" />
             </geometry>
         </collision>
-        <inertial>
-            <origin xyz="0 0 ${distance_shoulder_arm_z / 2}" rpy="0 0 0" />
+<inertial>
+            <origin rpy="0 0 0" xyz="0 0 0.04" />
             <mass value="0.8" />
-            <inertia ixx="0.0015" ixy="0.0" ixz="0.0" iyy="0.0015" iyz="0.0" izz="0.0015"/>
+            <inertia ixx="0.0015" ixy="0.0" ixz="0.0" iyy="0.0015" iyz="0.0" izz="0.0015" />
         </inertial>
     </link>
     <link name="arm_link">
         <visual>
-            <origin xyz="0 0 0" rpy="0 0 0" />
+            <origin rpy="0 0 0" xyz="0 0 0" />
             <geometry>
                 <mesh filename="package://niryo_one_description/meshes/v2/collada/arm_link.dae" />
@@ -88,18 +73,18 @@
         </visual>
         <collision>
-            <origin xyz="0 0 0" rpy="0 0 0" />
+            <origin rpy="0 0 0" xyz="0 0 0" />
             <geometry>
                 <mesh filename="package://niryo_one_description/meshes/v2/stl/arm_link.stl" />
             </geometry>
         </collision>
-        <inertial>
-            <origin xyz="${distance_arm_elbow_x / 2} -0.1 0" rpy="0 0 0" />
+<inertial>
+            <origin rpy="0 0 0" xyz="0.105 -0.1 0" />
             <mass value="0.4" />
-            <inertia ixx="0.0015" ixy="0.0" ixz="0.0" iyy="0.0015" iyz="0.0" izz="0.0015"/>
+            <inertia ixx="0.0015" ixy="0.0" ixz="0.0" iyy="0.0015" iyz="0.0" izz="0.0015" />
         </inertial>
     </link>
     <link name="elbow_link">
         <visual>
-            <origin xyz="0 0 0" rpy="0 0 0" />
+            <origin rpy="0 0 0" xyz="0 0 0" />
             <geometry>
                 <mesh filename="package://niryo_one_description/meshes/v2/collada/elbow_link.dae" />
@@ -107,18 +92,18 @@
         </visual>
         <collision>
-            <origin xyz="0 0 0" rpy="0 0 0" />
+            <origin rpy="0 0 0" xyz="0 0 0" />
             <geometry>
                 <mesh filename="package://niryo_one_description/meshes/v2/stl/elbow_link.stl" />
             </geometry>
         </collision>
-        <inertial>
-            <origin xyz="${distance_elbow_forearm_x / 2} ${distance_elbow_forearm_y / 2} 0" rpy="0 0 0" />
+<inertial>
+            <origin rpy="0 0 0" xyz="0.02075 0.015 0" />
             <mass value="0.3" />
-            <inertia ixx="0.0015" ixy="0.0" ixz="0.0" iyy="0.0015" iyz="0.0" izz="0.0015"/>
+            <inertia ixx="0.0015" ixy="0.0" ixz="0.0" iyy="0.0015" iyz="0.0" izz="0.0015" />
         </inertial>
     </link>
     <link name="forearm_link">
         <visual>
-            <origin xyz="0 0 0" rpy="0 0 0" />
+            <origin rpy="0 0 0" xyz="0 0 0" />
             <geometry>
                 <mesh filename="package://niryo_one_description/meshes/v2/collada/forearm_link.dae" />
@@ -126,18 +111,18 @@
         </visual>
         <collision>
-            <origin xyz="0 0 0" rpy="0 0 0" />
+            <origin rpy="0 0 0" xyz="0 0 0" />
             <geometry>
                 <mesh filename="package://niryo_one_description/meshes/v2/stl/forearm_link.stl" />
             </geometry>
         </collision>
-        <inertial>
-            <origin xyz="0 0 ${distance_forearm_wrist_z / 2}" rpy="0 0 0" />
+<inertial>
+            <origin rpy="0 0 0" xyz="0 0 0.09" />
             <mass value="0.3" />
-            <inertia ixx="0.0015" ixy="0.0" ixz="0.0" iyy="0.0015" iyz="0.0" izz="0.0015"/>
+            <inertia ixx="0.0015" ixy="0.0" ixz="0.0" iyy="0.0015" iyz="0.0" izz="0.0015" />
         </inertial>
     </link>
     <link name="wrist_link">
         <visual>
-            <origin xyz="0 0 0" rpy="0 0 0" />
+            <origin rpy="0 0 0" xyz="0 0 0" />
             <geometry>
                 <mesh filename="package://niryo_one_description/meshes/v2/collada/wrist_link.dae" />
@@ -145,18 +130,18 @@
         </visual>
         <collision>
-            <origin xyz="0 0 0" rpy="0 0 0" />
+            <origin rpy="0 0 0" xyz="0 0 0" />
             <geometry>
                 <mesh filename="package://niryo_one_description/meshes/v2/stl/wrist_link.stl" />
             </geometry>
         </collision>
-        <inertial>
-            <origin xyz="${distance_wrist_hand_x / 2} ${distance_wrist_hand_y / 2} 0" rpy="0 0 0" />
+<inertial>
+            <origin rpy="0 0 0" xyz="0.0082 -0.00275 0" />
             <mass value="0.15" />
-            <inertia ixx="0.001" ixy="0.0" ixz="0.0" iyy="0.001" iyz="0.0" izz="0.001"/>
+            <inertia ixx="0.001" ixy="0.0" ixz="0.0" iyy="0.001" iyz="0.0" izz="0.001" />
         </inertial>
     </link>
     <link name="hand_link">
         <visual>
-            <origin xyz="0 0 0" rpy="0 0 0" />
+            <origin rpy="0 0 0" xyz="0 0 0" />
             <geometry>
                 <mesh filename="package://niryo_one_description/meshes/v2/collada/hand_link.dae" />
@@ -164,29 +149,28 @@
         </visual>
         <collision>
-            <origin xyz="0 0 0" rpy="0 0 0" />
+            <origin rpy="0 0 0" xyz="0 0 0" />
             <geometry>
                 <mesh filename="package://niryo_one_description/meshes/v2/stl/hand_link.stl" />
             </geometry>
         </collision>
-        <inertial>
-            <origin xyz="0 0 ${distance_hand_tool / 2}" rpy="0 0 0" />
+<inertial>
+            <origin rpy="0 0 0" xyz="0 0 0.00365" />
             <mass value="0.05" />
-            <inertia ixx="0.001" ixy="0.0" ixz="0.0" iyy="0.001" iyz="0.0" izz="0.001"/>
-        </inertial>
-    </link>
-    <link name="tool_link">
-    </link>
+            <inertia ixx="0.001" ixy="0.0" ixz="0.0" iyy="0.001" iyz="0.0" izz="0.001" />
+        </inertial>
+    </link>
+    <link name="tool_link" />
     <!--Joints -->
     <joint name="joint_world" type="fixed">
-        <parent link="world"/>
-        <child link="base_link"/>
-        <origin xyz="0 0 0" rpy="0 0 0" />
+        <parent link="world" />
+        <child link="base_link" />
+        <origin rpy="0 0 0" xyz="0 0 0" />
     </joint>
     <joint name="joint_1" type="revolute">
         <parent link="base_link" />
         <child link="shoulder_link" />
-        <origin xyz="0 0 ${distance_origin_shoulder_z}" rpy="0 0 0" />
-        <axis xyz="0 0 1" />
-        <limit effort="100.0" velocity="3.0" lower="${limit_low_shoulder_rotation}" upper="${limit_up_shoulder_rotation}" />
+        <origin rpy="0 0 0" xyz="0 0 0.103" />
+        <axis xyz="0 0 1" />
+        <limit effort="100.0" lower="-3.05433" upper="3.05433" velocity="3.0" />
         <dynamics damping="0.1" friction="0.0" />
     </joint>
@@ -194,6 +178,6 @@
         <parent link="shoulder_link" />
         <child link="arm_link" />
-        <origin xyz="0 0 ${distance_shoulder_arm_z}" rpy="${PI/2} ${-PI/2} 0" />
-        <limit effort="100.0" velocity="3.0" lower="${limit_low_arm_rotation}" upper="${limit_up_arm_rotation}" />
+        <origin rpy="1.5707963268 -1.5707963268 0" xyz="0 0 0.08" />
+        <limit effort="100.0" lower="-1.91986" upper="0.640187" velocity="3.0" />
         <axis xyz="0 0 1" />
         <dynamics damping="0.1" friction="0.0" />
@@ -202,6 +186,6 @@
         <parent link="arm_link" />
         <child link="elbow_link" />
-        <origin xyz="${distance_arm_elbow_x} ${distance_arm_elbow_y} 0" rpy="0 0 ${-PI/2}" />
-        <limit effort="100.0" velocity="3.0" lower="${limit_low_elbow_rotation}" upper="${limit_up_elbow_rotation}" />
+        <origin rpy="0 0 -1.5707963268" xyz="0.21 0.0 0" />
+        <limit effort="100.0" lower="-1.397485" upper="1.5707963268" velocity="3.0" />
         <axis xyz="0 0 1" />
         <dynamics damping="0.1" friction="0.0" />
@@ -210,6 +194,6 @@
         <parent link="elbow_link" />
         <child link="forearm_link" />
-        <origin xyz="${distance_elbow_forearm_x} ${distance_elbow_forearm_y} 0" rpy="0 ${PI/2} 0" />
-        <limit effort="100.0" velocity="3.0" lower="${limit_low_forearm_rotation}" upper="${limit_up_forearm_rotation}" />
+        <origin rpy="0 1.5707963268 0" xyz="0.0415 0.03 0" />
+        <limit effort="100.0" lower="-3.05433" upper="3.05433" velocity="3.0" />
         <axis xyz="0 0 1" />
         <dynamics damping="0.1" friction="0.0" />
@@ -218,6 +202,6 @@
         <parent link="forearm_link" />
         <child link="wrist_link" />
-        <origin xyz="0 0 ${distance_forearm_wrist_z}" rpy="0 ${-PI/2} 0" />
-        <limit effort="100.0" velocity="3.0" lower="${limit_low_wrist_rotation}" upper="${limit_up_wrist_rotation}" />
+        <origin rpy="0 -1.5707963268 0" xyz="0 0 0.18" />
+        <limit effort="100.0" lower="-1.74533" upper="1.91986" velocity="3.0" />
         <axis xyz="0 0 1" />
         <dynamics damping="0.1" friction="0.0" />
@@ -226,6 +210,6 @@
         <parent link="wrist_link" />
         <child link="hand_link" />
-        <origin xyz="${distance_wrist_hand_x} ${distance_wrist_hand_y} 0" rpy="0 ${PI/2} 0" />
-        <limit effort="100.0" velocity="3.0" lower="${limit_low_hand_rotation}" upper="${limit_up_hand_rotation}" />
+        <origin rpy="0 1.5707963268 0" xyz="0.0164 -0.0055 0" />
+        <limit effort="100.0" lower="-2.57436" upper="2.57436" velocity="3.0" />
         <axis xyz="0 0 1" />
         <dynamics damping="0.1" friction="0.0" />
@@ -234,7 +218,7 @@
         <parent link="hand_link" />
         <child link="tool_link" />
-        <origin xyz="0 0 ${distance_hand_tool}" rpy="${-PI/2} ${-PI/2} 0" />
-    </joint>
-    <transmission name="transmission_1">
+        <origin rpy="-1.5707963268 -1.5707963268 0" xyz="0 0 0.0073" />
+    </joint>
+<transmission name="transmission_1">
         <type>transmission_interface/SimpleTransmission</type>
         <joint name="joint_1">
@@ -297,5 +281,7 @@
     </transmission>
     <gazebo>
-        <plugin name="gazebo_ros_control" filename="libgazebo_ros_control.so">
+        <plugin filename="libgazebo_ros_control.so" name="gazebo_ros_control">
+            <robotSimType>gazebo_ros_control/DefaultRobotHWSim</robotSimType>
+            <robotNamespace>/</robotNamespace>
         </plugin>
     </gazebo>
@@ -321,5 +307,124 @@
         <selfCollide>true</selfCollide>
     </gazebo>
-    <gazebo reference="tool_link">
-    </gazebo>
+    <gazebo reference="tool_link" />
+    <transmission name="trans_joint_1">
+        <type>transmission_interface/SimpleTransmission</type>
+        <joint name="joint_1">
+            <hardwareInterface>hardware_interface/EffortJointInterface</hardwareInterface>
+        </joint>
+        <actuator name="joint_1_motor">
+            <hardwareInterface>hardware_interface/EffortJointInterface</hardwareInterface>
+            <mechanicalReduction>1</mechanicalReduction>
+        </actuator>
+    </transmission>
+    <transmission name="trans_joint_2">
+        <type>transmission_interface/SimpleTransmission</type>
+        <joint name="joint_2">
+            <hardwareInterface>hardware_interface/EffortJointInterface</hardwareInterface>
+        </joint>
+        <actuator name="joint_2_motor">
+            <hardwareInterface>hardware_interface/EffortJointInterface</hardwareInterface>
+            <mechanicalReduction>1</mechanicalReduction>
+        </actuator>
+    </transmission>
+    <transmission name="trans_joint_3">
+        <type>transmission_interface/SimpleTransmission</type>
+        <joint name="joint_3">
+            <hardwareInterface>hardware_interface/EffortJointInterface</hardwareInterface>
+        </joint>
+        <actuator name="joint_3_motor">
+            <hardwareInterface>hardware_interface/EffortJointInterface</hardwareInterface>
+            <mechanicalReduction>1</mechanicalReduction>
+        </actuator>
+    </transmission>
+    <transmission name="trans_joint_4">
+        <type>transmission_interface/SimpleTransmission</type>
+        <joint name="joint_4">
+            <hardwareInterface>hardware_interface/EffortJointInterface</hardwareInterface>
+        </joint>
+        <actuator name="joint_4_motor">
+            <hardwareInterface>hardware_interface/EffortJointInterface</hardwareInterface>
+            <mechanicalReduction>1</mechanicalReduction>
+        </actuator>
+    </transmission>
+    <transmission name="trans_joint_5">
+        <type>transmission_interface/SimpleTransmission</type>
+        <joint name="joint_5">
+            <hardwareInterface>hardware_interface/EffortJointInterface</hardwareInterface>
+        </joint>
+        <actuator name="joint_5_motor">
+            <hardwareInterface>hardware_interface/EffortJointInterface</hardwareInterface>
+            <mechanicalReduction>1</mechanicalReduction>
+        </actuator>
+    </transmission>
+    <transmission name="trans_joint_6">
+        <type>transmission_interface/SimpleTransmission</type>
+        <joint name="joint_6">
+            <hardwareInterface>hardware_interface/EffortJointInterface</hardwareInterface>
+        </joint>
+        <actuator name="joint_6_motor">
+            <hardwareInterface>hardware_interface/EffortJointInterface</hardwareInterface>
+            <mechanicalReduction>1</mechanicalReduction>
+        </actuator>
+    </transmission>
+    <transmission name="trans_joint_1">
+        <type>transmission_interface/SimpleTransmission</type>
+        <joint name="joint_1">
+            <hardwareInterface>hardware_interface/PositionJointInterface</hardwareInterface>
+        </joint>
+        <actuator name="joint_1_motor">
+            <hardwareInterface>hardware_interface/PositionJointInterface</hardwareInterface>
+            <mechanicalReduction>1</mechanicalReduction>
+        </actuator>
+    </transmission>
+    <transmission name="trans_joint_2">
+        <type>transmission_interface/SimpleTransmission</type>
+        <joint name="joint_2">
+            <hardwareInterface>hardware_interface/PositionJointInterface</hardwareInterface>
+        </joint>
+        <actuator name="joint_2_motor">
+            <hardwareInterface>hardware_interface/PositionJointInterface</hardwareInterface>
+            <mechanicalReduction>1</mechanicalReduction>
+        </actuator>
+    </transmission>
+    <transmission name="trans_joint_3">
+        <type>transmission_interface/SimpleTransmission</type>
+        <joint name="joint_3">
+            <hardwareInterface>hardware_interface/PositionJointInterface</hardwareInterface>
+        </joint>
+        <actuator name="joint_3_motor">
+            <hardwareInterface>hardware_interface/PositionJointInterface</hardwareInterface>
+            <mechanicalReduction>1</mechanicalReduction>
+        </actuator>
+    </transmission>
+    <transmission name="trans_joint_4">
+        <type>transmission_interface/SimpleTransmission</type>
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