Commit message: create launch file for Niryo with gripper support

File: niryo_one_description/urdf/v2/gazebo_niryo_one.urdf.xacro (robot description, xacro)
@@ -1,7 +1,3 @@
 <?xml version="1.0" encoding="utf-8" ?>
-<!-- =================================================================================== -->
-<!-- |    This document was autogenerated by xacro from /home/wolf/ros_ws/src/test_niryo_moveit/n1_description/urdf/gazebo_niryo_one.urdf.xacro | -->
-<!-- |    EDITING THIS FILE BY HAND IS NOT RECOMMENDED                                 | -->
-<!-- =================================================================================== -->
 <!-- =================================================================================== -->
 <!-- |    This document was autogenerated by xacro from /home/wolf/ros_ws/src/test_niryo_moveit/n1_description/urdf/gazebo_niryo_one.urdf.xacro | -->
@@ -220,64 +216,4 @@
         <origin rpy="-1.5707963268 -1.5707963268 0" xyz="0 0 0.0073" />
     </joint>
-<transmission name="transmission_1">
-        <type>transmission_interface/SimpleTransmission</type>
-        <joint name="joint_1">
-            <hardwareInterface>hardware_interface/EffortJointInterface</hardwareInterface>
-        </joint>
-        <actuator name="motor_1">
-            <hardwareInterface>hardware_interface/EffortJointInterface</hardwareInterface>
-            <mechanicalReduction>1</mechanicalReduction>
-        </actuator>
-    </transmission>
-    <transmission name="transmission_2">
-        <type>transmission_interface/SimpleTransmission</type>
-        <joint name="joint_2">
-            <hardwareInterface>hardware_interface/EffortJointInterface</hardwareInterface>
-        </joint>
-        <actuator name="motor_2">
-            <hardwareInterface>hardware_interface/EffortJointInterface</hardwareInterface>
-            <mechanicalReduction>1</mechanicalReduction>
-        </actuator>
-    </transmission>
-    <transmission name="transmission_3">
-        <type>transmission_interface/SimpleTransmission</type>
-        <joint name="joint_3">
-            <hardwareInterface>hardware_interface/EffortJointInterface</hardwareInterface>
-        </joint>
-        <actuator name="motor_3">
-            <hardwareInterface>hardware_interface/EffortJointInterface</hardwareInterface>
-            <mechanicalReduction>1</mechanicalReduction>
-        </actuator>
-    </transmission>
-    <transmission name="transmission_4">
-        <type>transmission_interface/SimpleTransmission</type>
-        <joint name="joint_4">
-            <hardwareInterface>hardware_interface/EffortJointInterface</hardwareInterface>
-        </joint>
-        <actuator name="motor_4">
-            <hardwareInterface>hardware_interface/EffortJointInterface</hardwareInterface>
-            <mechanicalReduction>1</mechanicalReduction>
-        </actuator>
-    </transmission>
-    <transmission name="transmission_5">
-        <type>transmission_interface/SimpleTransmission</type>
-        <joint name="joint_5">
-            <hardwareInterface>hardware_interface/EffortJointInterface</hardwareInterface>
-        </joint>
-        <actuator name="motor_5">
-            <hardwareInterface>hardware_interface/EffortJointInterface</hardwareInterface>
-            <mechanicalReduction>1</mechanicalReduction>
-        </actuator>
-    </transmission>
-    <transmission name="transmission_6">
-        <type>transmission_interface/SimpleTransmission</type>
-        <joint name="joint_6">
-            <hardwareInterface>hardware_interface/EffortJointInterface</hardwareInterface>
-        </joint>
-        <actuator name="motor_6">
-            <hardwareInterface>hardware_interface/EffortJointInterface</hardwareInterface>
-            <mechanicalReduction>1</mechanicalReduction>
-        </actuator>
-    </transmission>
     <gazebo>
         <plugin filename="libgazebo_ros_control.so" name="gazebo_ros_control">

File: niryo_one_description/urdf/v2/gripper.urdf.xacro (robot description, xacro)
@@ -1,3 +1,4 @@
 <robot xmlns:xacro="http://ros.org/wiki/xacro" name="gripper">
+    <xacro:include filename="$(find niryo_one_description)/urdf/v2/gazebo_niryo_one.urdf.xacro"/>
     <xacro:property name="PI" value="3.14159265359"/>
     <!-- Transmission macro -->
@@ -23,9 +24,9 @@
         </plugin>
     </gazebo>
-    <link name="world" />
+    <!-- <link name="world" /> -->
     <!-- <link name="base_link"> -->
     <!-- Joint from tool_link to base_gripper -->
     <joint name="joint_to_gripper" type="fixed">
-        <parent link="world"/>
+        <parent link="tool_link"/>
         <child link="base_gripper_1"/>
         <origin
